Commit message: created pybullet wrapper for iiwa + cmakelists changes + added tennisball endeffector in urdf

File: urdf/iiwa.urdf (robot description, URDF)
Before this commit: robot KUKAiiwa14, 8 links, 7 joints
Links:
- added link contact, mass 0.057; collision mesh filename=package://robot_properties_iiwa/meshes/sphere.obj scale=0.065 0.065 0.065; visual mesh filename=package://robot_properties_iiwa/meshes/sphere.obj scale=0.065 0.065 0.065
- link L1: geometry visual mesh filename=package://robot_properties_iiwa/meshes/iiwa14_link1.stl scale=0.001 0.001 0.001
- link L2: geometry visual mesh filename=package://robot_properties_iiwa/meshes/iiwa14_link2.stl scale=0.001 0.001 0.001
- link L3: geometry visual mesh filename=package://robot_properties_iiwa/meshes/iiwa14_link3.stl scale=0.001 0.001 0.001
- link L4: geometry visual mesh filename=package://robot_properties_iiwa/meshes/iiwa14_link4.stl scale=0.001 0.001 0.001
- link L5: geometry visual mesh filename=package://robot_properties_iiwa/meshes/iiwa14_link5.stl scale=0.001 0.001 0.001
- link L6: geometry visual mesh filename=package://robot_properties_iiwa/meshes/iiwa14_link6.stl scale=0.001 0.001 0.001
- link L7: geometry visual mesh filename=package://robot_properties_iiwa/meshes/iiwa14_link7.stl scale=0.001 0.001 0.001
- link iiwaBase: mass None -> 4.00000; geometry visual mesh filename=package://robot_properties_iiwa/meshes/iiwa14_base.stl scale=0.001 0.001 0.001
Joints:
- added joint END: type fixed, parent L7, child contact, origin xyz=0 0.0 0.04 rpy=0 0 0, limit lower=-10 upper=10 effort=1000 velocity=1000

Commit message: updated .gitignore + added demo script + updated urdf + updated CMakeLists + updated config.py

File: urdf/iiwa.urdf (robot description, URDF)
Before this commit: robot KUKAiiwa14, 9 links, 8 joints
Links:
- link iiwaBase: mass 4.00000 -> 8.00000
