Commit message: updated following new robot_properties_solo template . Added xacro and srdf . Still need debug

File: src/robot_properties_kuka/resources/urdf/iiwa.urdf (robot description, URDF)
Before this commit: robot KUKAiiwa14, 9 links, 8 joints
Links:
- removed link iiwaBase
- added link iiwa14_base, mass 8.00000; visual mesh filename=package://robot_properties_kuka/meshes/stl/iiwa14_base.stl scale=0.001 0.001 0.001
- link L1: geometry visual mesh filename=package://robot_properties_kuka/meshes/stl/iiwa14_link1.stl scale=0.001 0.001 0.001
- link L2: geometry visual mesh filename=package://robot_properties_kuka/meshes/stl/iiwa14_link2.stl scale=0.001 0.001 0.001
- link L3: geometry visual mesh filename=package://robot_properties_kuka/meshes/stl/iiwa14_link3.stl scale=0.001 0.001 0.001
- link L4: geometry visual mesh filename=package://robot_properties_kuka/meshes/stl/iiwa14_link4.stl scale=0.001 0.001 0.001
- link L5: geometry visual mesh filename=package://robot_properties_kuka/meshes/stl/iiwa14_link5.stl scale=0.001 0.001 0.001
- link L6: geometry visual mesh filename=package://robot_properties_kuka/meshes/stl/iiwa14_link6.stl scale=0.001 0.001 0.001
- link L7: geometry visual mesh filename=package://robot_properties_kuka/meshes/stl/iiwa14_link7.stl scale=0.001 0.001 0.001
- link contact: geometry collision mesh filename=package://robot_properties_kuka/meshes/sphere.obj scale=0.065 0.065 0.065; visual mesh filename=package://robot_properties_kuka/meshes/sphere.obj scale=0.065 0.065 0.065
Joints:
- joint A1: parent iiwaBase -> iiwa14_base
