Commit message: fixed xacro and urdf + stl names and some bugs in iiwaWrapper

File: src/robot_properties_kuka/resources/pre_generated_urdf/iiwa.urdf (robot description, URDF)
Before this commit: robot KUKAiiwa14, 9 links, 8 joints
Links:
- removed link iiwa14_base
- added link iiwa_base, mass 8.00000; visual mesh filename=package://meshes/stl/iiwa_base.stl scale=0.001 0.001 0.001
- link L1: mass 4.00000 -> 3.94781; geometry visual mesh filename=package://meshes/stl/iiwa_link1.stl scale=0.001 0.001 0.001
- link L2: geometry visual mesh filename=package://meshes/stl/iiwa_link2.stl scale=0.001 0.001 0.001
- link L3: geometry visual mesh filename=package://meshes/stl/iiwa_link3.stl scale=0.001 0.001 0.001
- link L4: geometry visual mesh filename=package://meshes/stl/iiwa_link4.stl scale=0.001 0.001 0.001
- link L5: geometry visual mesh filename=package://meshes/stl/iiwa_link5.stl scale=0.001 0.001 0.001
- link L6: geometry visual mesh filename=package://meshes/stl/iiwa_link6.stl scale=0.001 0.001 0.001
- link L7: geometry visual mesh filename=package://meshes/stl/iiwa_link7.stl scale=0.001 0.001 0.001
- link contact: geometry collision mesh filename=package://meshes/sphere.obj scale=0.065 0.065 0.065; visual mesh filename=package://meshes/sphere.obj scale=0.065 0.065 0.065
Joints:
- removed joint END
- added joint A0: type fixed, parent world, child iiwa_base, origin xyz=0.0 0.0 0.0 rpy=0.0 0.0 0.0
- added joint EE: type fixed, parent L7, child contact, origin xyz=0 0.0 0.04 rpy=0 0 0, limit lower=-10 upper=10 effort=1000 velocity=1000
- joint A1: limit effort=30 velocity=1.0 -> lower=-2.96706 upper=2.96706 effort=320 velocity=1.48353; parent iiwa14_base -> iiwa_base
- joint A2: limit effort=30 velocity=1.0 -> lower=-2.0944 upper=2.0944 effort=320 velocity=1.48353
- joint A3: limit effort=30 velocity=1.0 -> lower=-2.96706 upper=2.96706 effort=176 velocity=1.74533
- joint A4: limit effort=30 velocity=1.0 -> lower=-2.0944 upper=2.0944 effort=176 velocity=1.309
- joint A5: limit effort=30 velocity=1.0 -> lower=-2.96706 upper=2.96706 effort=110 velocity=2.26893
- joint A6: limit effort=30 velocity=1.0 -> lower=-2.0944 upper=2.0944 effort=40 velocity=2.35619
- joint A7: limit effort=30 velocity=1.0 -> lower=-3.05433 upper=3.05433 effort=40 velocity=2.35619

File: src/robot_properties_kuka/resources/xacro/iiwa.xacro (robot description, xacro)
@@ -10,16 +10,14 @@
   <xacro:property name="safety_controller_k_pos" value="100" />
   <xacro:property name="safety_controller_k_vel" value="2" />
-  <xacro:property name="joint_damping" value="0.5" />
-  <xacro:property name="max_effort" value="300"/>
-  <xacro:property name="max_velocity" value="10"/>
+  <xacro:property name="joint_damping" value="0.0" />
   <xacro:macro name="KUKAiiwa14" params="parent hardware_interface robot_name *origin">
     <!--joint between {parent} and base-->
-    <joint name="${parent}_KUKAiiwa14_joint" type="fixed">
+    <joint name="${parent}_joint" type="fixed">
       <xacro:insert_block name="origin"/>
       <parent link="${parent}"/>
-      <child link="KUKAiiwa14_base"/>
+      <child link="iiwa_base"/>
     </joint>
     <!-- BASE -->
-    <link name="KUKAiiwa14_base">
+    <link name="iiwa_base">
       <inertial>
         <origin xyz="-0.1 0 0.07" rpy="0 0 0"/>
@@ -30,5 +28,5 @@
         <origin xyz="0 0 0" rpy="0 0 0"/>
         <geometry>
-          <mesh filename="package://meshes/stl/iiwa14_base.stl"/>
+          <mesh filename="package://meshes/stl/iiwa_base.stl"/>
         </geometry>
         <material name="Grey"/>
@@ -37,5 +35,5 @@
         <origin xyz="0 0 0" rpy="0 0 0"/>
         <geometry>
-          <mesh filename="package://meshes/stl/iiwa14_base.stl"/>
+          <mesh filename="package://meshes/stl/iiwa_base.stl"/>
         </geometry>
         <material name="Grey"/>
@@ -49,11 +47,10 @@
     </link>
     <!-- joint between base and link1 -->
-    <joint name="KUKAiiwa14_joint_1" type="revolute">
-      <parent link="KUKAiiwa14_base"/>
-      <child link="KUKAiiwa14_link1"/>
+    <joint name="A1" type="revolute">
+      <parent link="iiwa_base"/>
+      <child link="L1"/>
       <origin xyz="0 0 0.1575" rpy="0 0 0"/>
       <axis xyz="0 0 1"/>
-      <limit lower="${-170 * PI / 180}" upper="${170 * PI / 180}"
-             effort="${max_effort}" velocity="${max_velocity}" />
+      <limit lower="-2.96706" upper="2.96706" velocity="1.48353" effort="320"/>
       <safety_controller soft_lower_limit="${-168 * PI / 180}"
                          soft_upper_limit="${168 * PI / 180}"
@@ -63,5 +60,5 @@
     </joint>
     <!-- LINK 1-->
-    <link name="KUKAiiwa14_link1">
+    <link name="L1">
       <inertial>
         <origin xyz="0 -0.03 0.12" rpy="0 0 0"/>
@@ -72,12 +69,12 @@
         <origin xyz="0 0 0" rpy="0 0 0"/>
         <geometry>
-          <mesh filename="package://meshes/stl/iiwa14_link1.stl"/>
-        </geometry>
-        <material name="Orange"/>
-      </visual>
-      <collision>
-        <origin xyz="0 0 0" rpy="0 0 0"/>
-        <geometry>
-          <mesh filename="package://meshes/stl/iiwa14_link1.stl"/>
+          <mesh filename="package://meshes/stl/iiwa_link_1.stl"/>
+        </geometry>
+        <material name="Orange"/>
+      </visual>
+      <collision>
+        <origin xyz="0 0 0" rpy="0 0 0"/>
+        <geometry>
+          <mesh filename="package://meshes/stl/iiwa_link_1.stl"/>
         </geometry>
         <material name="Orange"/>
@@ -85,11 +82,10 @@
     </link>
     <!-- joint between link1 and link2 -->
-    <joint name="KUKAiiwa14_joint_2" type="revolute">
-      <parent link="KUKAiiwa14_link1"/>
-      <child link="KUKAiiwa14_link2"/>
+    <joint name="A2" type="revolute">
+      <parent link="L1"/>
+      <child link="L2"/>
       <origin xyz="0 0 0.2025" rpy="${PI / 2}   0 ${PI}"/>
       <axis xyz="0 0 1"/>
-      <limit lower="${-120 * PI / 180}" upper="${120 * PI / 180}"
-             effort="${max_effort}" velocity="${max_velocity}" />
+      <limit lower="-2.0944" upper="2.0944" velocity="1.48353" effort="320"/>
       <safety_controller soft_lower_limit="${-118 * PI / 180}"
                          soft_upper_limit="${118 * PI / 180}"
@@ -99,5 +95,5 @@
     </joint>
     <!-- LINK 2-->
-    <link name="KUKAiiwa14_link2">
+    <link name="L2">
       <inertial>
         <origin xyz="0.0003 0.059 0.042" rpy="0 0 0"/>
@@ -108,12 +104,12 @@
         <origin xyz="0 0 0" rpy="0 0 0"/>
         <geometry>
-          <mesh filename="package://meshes/stl/iiwa14_link2.stl"/>
-        </geometry>
-        <material name="Orange"/>
-      </visual>
-      <collision>
-        <origin xyz="0 0 0" rpy="0 0 0"/>
-        <geometry>
-          <mesh filename="package://meshes/stl/iiwa14_link2.stl"/>
+          <mesh filename="package://meshes/stl/iiwa_link_2.stl"/>
+        </geometry>
+        <material name="Orange"/>
+      </visual>
+      <collision>
+        <origin xyz="0 0 0" rpy="0 0 0"/>
+        <geometry>
+          <mesh filename="package://meshes/stl/iiwa_link_2.stl"/>
         </geometry>
         <material name="Orange"/>
@@ -121,11 +117,10 @@
     </link>
     <!-- joint between link2 and link3 -->
-    <joint name="KUKAiiwa14_joint_3" type="revolute">
-      <parent link="KUKAiiwa14_link2"/>
-      <child link="KUKAiiwa14_link3"/>
+    <joint name="A3" type="revolute">
+      <parent link="L2"/>
+      <child link="L3"/>
       <origin xyz="0 0.2045 0" rpy="${PI / 2} 0 ${PI}"/>
       <axis xyz="0 0 1"/>
-      <limit lower="${-170 * PI / 180}" upper="${170 * PI / 180}"
-             effort="${max_effort}" velocity="${max_velocity}" />
+      <limit lower="-2.96706" upper="2.96706" velocity="1.74533" effort="176"/>
       <safety_controller soft_lower_limit="${-168 * PI / 180}"
                          soft_upper_limit="${168 * PI / 180}"
@@ -135,5 +130,5 @@
     </joint>
     <!-- LINK 3-->
-    <link name="KUKAiiwa14_link3">
+    <link name="L3">
       <inertial>
         <origin xyz="0 0.03 0.13" rpy="0 0 0"/>
@@ -144,12 +139,12 @@
         <origin xyz="0 0 0" rpy="0 0 0"/>
         <geometry>
-          <mesh filename="package://meshes/stl/iiwa14_link3.stl"/>
-        </geometry>
-        <material name="Orange"/>
-      </visual>
-      <collision>
-        <origin xyz="0 0 0" rpy="0 0 0"/>
-        <geometry>
-          <mesh filename="package://meshes/stl/iiwa14_link3.stl"/>
+          <mesh filename="package://meshes/stl/iiwa_link_3.stl"/>
+        </geometry>
+        <material name="Orange"/>
+      </visual>
+      <collision>
+        <origin xyz="0 0 0" rpy="0 0 0"/>
+        <geometry>
+          <mesh filename="package://meshes/stl/iiwa_link_3.stl"/>
         </geometry>
         <material name="Orange"/>
@@ -157,11 +152,10 @@
     </link>
     <!-- joint between link3 and link4 -->
-    <joint name="KUKAiiwa14_joint_4" type="revolute">
-      <parent link="KUKAiiwa14_link3"/>
-      <child link="KUKAiiwa14_link4"/>
+    <joint name="A4" type="revolute">
+      <parent link="L3"/>
+      <child link="L4"/>
       <origin xyz="0 0 0.2155" rpy="${PI / 2} 0 0"/>
       <axis xyz="0 0 1"/>
-      <limit lower="${-120 * PI / 180}" upper="${120 * PI / 180}"
-             effort="${max_effort}" velocity="${max_velocity}" />
+      <limit lower="-2.0944" upper="2.0944" velocity="1.309" effort="176"/>
       <safety_controller soft_lower_limit="${-118 * PI / 180}"
                          soft_upper_limit="${118 * PI / 180}"
@@ -171,5 +165,5 @@
     </joint>
     <!-- LINK 4-->
-    <link name="KUKAiiwa14_link4">
+    <link name="L4">
       <inertial>
         <origin xyz="0 0.067 0.034" rpy="0 0 0"/>
@@ -180,12 +174,12 @@
         <origin xyz="0 0 0" rpy="0 0 0"/>
         <geometry>
-          <mesh filename="package://meshes/stl/iiwa14_link4.stl"/>
-        </geometry>
-        <material name="Orange"/>
-      </visual>
-      <collision>
-        <origin xyz="0 0 0" rpy="0 0 0"/>
-        <geometry>
-          <mesh filename="package://meshes/stl/iiwa14_link4.stl"/>
+          <mesh filename="package://meshes/stl/iiwa_link_4.stl"/>
+        </geometry>
+        <material name="Orange"/>
+      </visual>
+      <collision>
+        <origin xyz="0 0 0" rpy="0 0 0"/>
+        <geometry>
+          <mesh filename="package://meshes/stl/iiwa_link_4.stl"/>
         </geometry>
         <material name="Orange"/>
@@ -193,11 +187,10 @@
     </link>
     <!-- joint between link4 and link5 -->
-    <joint name="KUKAiiwa14_joint_5" type="revolute">
-      <parent link="KUKAiiwa14_link4"/>
-      <child link="KUKAiiwa14_link5"/>
+    <joint name="A5" type="revolute">
+      <parent link="L4"/>
+      <child link="L5"/>
       <origin xyz="0 0.1845 0" rpy="${-PI / 2} ${PI} 0"/>
       <axis xyz="0 0 1"/>
-      <limit lower="${-170 * PI / 180}" upper="${170 * PI / 180}"
-             effort="${max_effort}" velocity="${max_velocity}" />
+      <limit lower="-2.96706" upper="2.96706" velocity="2.26893" effort="110"/>
       <safety_controller soft_lower_limit="${-168 * PI / 180}"
                          soft_upper_limit="${168 * PI / 180}"
@@ -207,5 +200,5 @@
     </joint>
     <!-- LINK 5-->
-    <link name="KUKAiiwa14_link5">
+    <link name="L5">
       <inertial>
         <origin xyz="0.0001 0.021 0.076" rpy="0 0 0"/>
@@ -216,12 +209,12 @@
         <origin xyz="0 0 0" rpy="0 0 0"/>
         <geometry>
-          <mesh filename="package://meshes/stl/iiwa14_link5.stl"/>
-        </geometry>
-        <material name="Orange"/>
-      </visual>
-      <collision>
-        <origin xyz="0 0 0" rpy="0 0 0"/>
-        <geometry>
-          <mesh filename="package://meshes/stl/iiwa14_link5.stl"/>
+          <mesh filename="package://meshes/stl/iiwa_link_5.stl"/>
+        </geometry>
+        <material name="Orange"/>
+      </visual>
+      <collision>
+        <origin xyz="0 0 0" rpy="0 0 0"/>
+        <geometry>
+          <mesh filename="package://meshes/stl/iiwa_link_5.stl"/>
         </geometry>
         <material name="Orange"/>
@@ -229,11 +222,10 @@
     </link>
     <!-- joint between link5 and link6 -->
-    <joint name="KUKAiiwa14_joint_6" type="revolute">
-      <parent link="KUKAiiwa14_link5"/>
-      <child link="KUKAiiwa14_link6"/>
+    <joint name="A6" type="revolute">
+      <parent link="L5"/>
+      <child link="L6"/>
       <origin xyz="0 0 0.2155" rpy="${PI / 2} 0 0"/>
       <axis xyz="0 0 1"/>
-      <limit lower="${-120 * PI / 180}" upper="${120 * PI / 180}"
-             effort="${max_effort}" velocity="${max_velocity}" />
+      <limit lower="-2.0944" upper="2.0944" velocity="2.35619" effort="40"/>
       <safety_controller soft_lower_limit="${-118 * PI / 180}"
                          soft_upper_limit="${118 * PI / 180}"
@@ -243,5 +235,5 @@
     </joint>
     <!-- LINK 6-->
-    <link name="KUKAiiwa14_link6">
+    <link name="L6">
       <inertial>
         <origin xyz="0 0.0006 0.0004" rpy="0 0 0"/>
@@ -252,12 +244,12 @@
         <origin xyz="0 0 0" rpy="0 0 0"/>
         <geometry>
-          <mesh filename="package://meshes/stl/iiwa14_link6.stl"/>
-        </geometry>
-        <material name="Orange"/>
-      </visual>
-      <collision>
-        <origin xyz="0 0 0" rpy="0 0 0"/>
-        <geometry>
-          <mesh filename="package://meshes/stl/iiwa14_link6.stl"/>
+          <mesh filename="package://meshes/stl/iiwa_link_6.stl"/>
+        </geometry>
+        <material name="Orange"/>
+      </visual>
+      <collision>
+        <origin xyz="0 0 0" rpy="0 0 0"/>
+        <geometry>
+          <mesh filename="package://meshes/stl/iiwa_link_6.stl"/>
         </geometry>
         <material name="Orange"/>
@@ -265,11 +257,10 @@
     </link>
     <!-- joint between link6 and link7 -->
-    <joint name="KUKAiiwa14_joint_7" type="revolute">
-      <parent link="KUKAiiwa14_link6"/>
-      <child link="KUKAiiwa14_link7"/>
+    <joint name="A7" type="revolute">
+      <parent link="L6"/>
+      <child link="L7"/>
       <origin xyz="0 0.081 0" rpy="${- PI / 2} ${PI} 0"/>
       <axis xyz="0 0 1"/>
-      <limit lower="${-175 * PI / 180}" upper="${175 * PI / 180}"
-             effort="${max_effort}" velocity="${max_velocity}" />
+      <limit lower="-3.05433" upper="3.05433" velocity="2.35619" effort="40" />
       <safety_controller soft_lower_limit="${-173 * PI / 180}"
                          soft_upper_limit="${173 * PI / 180}"
@@ -279,5 +270,5 @@
     </joint>
     <!-- LINK 7-->
-    <link name="KUKAiiwa14_link7">
+    <link name="L7">
       <inertial>
         <origin xyz="0 0 0.02" rpy="0 0 0"/>
@@ -288,5 +279,5 @@
         <origin xyz="0 0 0" rpy="0 0 0"/>
         <geometry>
-          <mesh filename="package://meshes/stl/iiwa14_link7.stl"/>
+          <mesh filename="package://meshes/stl/iiwa_link_7.stl"/>
         </geometry>
         <material name="Grey"/>
@@ -295,16 +286,51 @@
         <origin xyz="0 0 0" rpy="0 0 0"/>
         <geometry>
-          <mesh filename="package://meshes/stl/iiwa14_link7.stl"/>
+          <mesh filename="package://meshes/stl/iiwa_link_7.stl"/>
         </geometry>
         <material name="Grey"/>
       </collision>
     </link>
-    <joint name="KUKAiiwa14_joint_ee" type="fixed">
-      <parent link="KUKAiiwa14_link7"/>
-      <child link="contact"/>
-      <origin xyz="0 0 0.045" rpy="0 0 0"/>
-    </joint>
-    <link name="contact">
-    </link>
+  <!-- EE -->
+  <joint name="EE" type="fixed">
+    <parent link="L7"/>
+    <child link="contact"/>
+    <!-- Joint placement -->
+    <origin rpy="0 0 0" xyz="0 0.0 0.04"/>
+    <!-- Limits (usefull?) -->
+    <limit effort="1000" lower="-10" upper="10" velocity="1000"/>
+    <!-- pybullet simulation parameters -->
+    <dynamics damping="0.0" friction="0.0"/>
+  </joint>
+  <!-- CONTACT (modeled by a tennis ball) -->
+  <link name="contact">
+    <inertial>
+      <origin rpy="0 0 0" xyz="0 0 0.0"/>
+      <mass value="0.057"/>
+      <inertia ixx="0.0000354" ixy="0.0" ixz="0.0" iyy="0.0000354" iyz="0.0" izz="0.0000354"/>
+    </inertial>
+    <visual>
+      <origin rpy="0 0 0" xyz="0 0 0"/>
+      <geometry>
+        <mesh filename="package://meshes/sphere.obj" scale="0.065 0.065 0.065"/>/>
+      </geometry>
+      <material name="grey">
+        <color rgba="0.8 0.8 0.8 1.0"/>
+      </material>
+    </visual>
+    <collision>
+      <origin rpy="0 0 0" xyz="0 0 0"/>
+      <geometry>
+        <mesh filename="package://meshes/sphere.obj" scale="0.065 0.065 0.065"/>/>
+      </geometry>
+      <material name="grey">
+        <color rgba="0.8 0.8 0.8 1.0"/>
+      </material>
+    </collision>
+    <!-- Bullet specific paramters -->
+    <contact>
+      <lateral_friction value="1.0"/>
+      <restitution value="0.5"/>
+    </contact>
+  </link>
     <!--Extensions -->
     <xacro:iiwa_gazebo robot_name="KUKAiiwa14" />
