Commit message: fixed problem with bullet_utils

File: src/robot_properties_kuka/resources/pre_generated_urdf/iiwa.urdf (robot description, URDF)
Before this commit: robot KUKAiiwa, 9 links, 9 joints
Links:
- link L1: mass 3.94781 -> 4.00000; geometry visual mesh filename=package://meshes/stl/iiwa_link_1.stl scale=0.001 0.001 0.001
- link L2: geometry visual mesh filename=package://meshes/stl/iiwa_link_2.stl scale=0.001 0.001 0.001
- link L3: geometry visual mesh filename=package://meshes/stl/iiwa_link_3.stl scale=0.001 0.001 0.001
- link L4: geometry visual mesh filename=package://meshes/stl/iiwa_link_4.stl scale=0.001 0.001 0.001
- link L5: geometry visual mesh filename=package://meshes/stl/iiwa_link_5.stl scale=0.001 0.001 0.001
- link L6: geometry visual mesh filename=package://meshes/stl/iiwa_link_6.stl scale=0.001 0.001 0.001
- link L7: geometry visual mesh filename=package://meshes/stl/iiwa_link_7.stl scale=0.001 0.001 0.001
- link contact: geometry 
Joints:
- removed joint A0
- joint A1: limit lower=-2.96706 upper=2.96706 effort=320 velocity=1.48353 -> effort=30 velocity=1.0
- joint A2: limit lower=-2.0944 upper=2.0944 effort=320 velocity=1.48353 -> effort=30 velocity=1.0
- joint A3: limit lower=-2.96706 upper=2.96706 effort=176 velocity=1.74533 -> effort=30 velocity=1.0
- joint A4: limit lower=-2.0944 upper=2.0944 effort=176 velocity=1.309 -> effort=30 velocity=1.0
- joint A5: limit lower=-2.96706 upper=2.96706 effort=110 velocity=2.26893 -> effort=30 velocity=1.0
- joint A6: limit lower=-2.0944 upper=2.0944 effort=40 velocity=2.35619 -> effort=30 velocity=1.0
- joint A7: limit lower=-3.05433 upper=3.05433 effort=40 velocity=2.35619 -> effort=30 velocity=1.0

File: src/robot_properties_kuka/resources/xacro/iiwa.urdf.xacro (robot description, xacro)
@@ -6,5 +6,5 @@
   <xacro:include filename="iiwa.xacro"/>
   <!-- Fix to world just for testing -->
-  <link name="world"/>
+  <!-- <link name="world"/> -->
   <!--KUKAiiwa14-->
   <xacro:KUKAiiwa14 hardware_interface="PositionJointInterface" robot_name="KUKAiiwa14" parent="world">

File: src/robot_properties_kuka/resources/xacro/iiwa.xacro (robot description, xacro)
@@ -2,9 +2,9 @@
 <robot xmlns:xacro="http://www.ros.org/wiki/xacro">
   <!-- Import all Gazebo-customization elements, including Gazebo colors -->
-  <xacro:include filename="iiwa.gazebo.xacro" />
+  <!-- <xacro:include filename="iiwa.gazebo.xacro" /> -->
   <!-- Import Transmissions -->
-  <xacro:include filename="iiwa.transmission.xacro" />
+  <!-- <xacro:include filename="iiwa.transmission.xacro" /> -->
   <!-- Include Utilities -->
-  <xacro:include filename="utilities.xacro" />
+  <!-- <xacro:include filename="utilities.xacro" /> -->
   <!-- some constants -->
   <xacro:property name="safety_controller_k_pos" value="100" />
@@ -12,14 +12,15 @@
   <xacro:property name="joint_damping" value="0.0" />
   <xacro:macro name="KUKAiiwa14" params="parent hardware_interface robot_name *origin">
-    <!--joint between {parent} and base-->
-    <joint name="${parent}_joint" type="fixed">
+    <!--joint between WORLD and BASE-->
+    <!-- <joint name="A0" type="fixed">
       <xacro:insert_block name="origin"/>
-      <parent link="${parent}"/>
+      <parent link="world"/>
       <child link="iiwa_base"/>
     </joint>
+     -->
     <!-- BASE -->
     <link name="iiwa_base">
       <inertial>
-        <origin xyz="-0.1 0 0.07" rpy="0 0 0"/>
+        <origin xyz="0 0 0" rpy="0 0 0"/>
         <mass value="5"/>
         <inertia ixx="0.05"  ixy="0"  ixz="0" iyy="0.06" iyz="0" izz="0.03" />
@@ -28,5 +29,5 @@
         <origin xyz="0 0 0" rpy="0 0 0"/>
         <geometry>
-          <mesh filename="package://meshes/stl/iiwa_base.stl"/>
+          <mesh filename="package://meshes/stl/iiwa_base.stl" scale="0.001 0.001 0.001"/>
         </geometry>
         <material name="Grey"/>
@@ -35,5 +36,5 @@
         <origin xyz="0 0 0" rpy="0 0 0"/>
         <geometry>
-          <mesh filename="package://meshes/stl/iiwa_base.stl"/>
+          <mesh filename="package://meshes/stl/iiwa_base.stl" scale="0.001 0.001 0.001"/>
         </geometry>
         <material name="Grey"/>
@@ -62,19 +63,19 @@
     <link name="L1">
       <inertial>
-        <origin xyz="0 -0.03 0.12" rpy="0 0 0"/>
-        <mass value="4"/>
-        <inertia ixx="0.1"  ixy="0"  ixz="0" iyy="0.09" iyz="0" izz="0.02" />
-      </inertial>
-      <visual>
-        <origin xyz="0 0 0" rpy="0 0 0"/>
-        <geometry>
-          <mesh filename="package://meshes/stl/iiwa_link_1.stl"/>
-        </geometry>
-        <material name="Orange"/>
-      </visual>
-      <collision>
-        <origin xyz="0 0 0" rpy="0 0 0"/>
-        <geometry>
-          <mesh filename="package://meshes/stl/iiwa_link_1.stl"/>
+        <origin xyz="0.00000 0.00000 0.00000"/>
+        <mass value="3.94781"/>
+        <inertia ixx="0.00455" iyy="0.00454" izz="0.00029" ixy="0.00000" ixz="-0.00000" iyz="-0.00001"/>
+      </inertial>
+      <visual>
+        <origin xyz="0 0 0" rpy="0 0 0"/>
+        <geometry>
+          <mesh filename="package://meshes/stl/iiwa_link_1.stl" scale="0.001 0.001 0.001"/>
+        </geometry>
+        <material name="Orange"/>
+      </visual>
+      <collision>
+        <origin xyz="0 0 0" rpy="0 0 0"/>
+        <geometry>
+          <mesh filename="package://meshes/stl/iiwa_link_1.stl" scale="0.001 0.001 0.001"/>
         </geometry>
         <material name="Orange"/>
@@ -104,12 +105,12 @@
         <origin xyz="0 0 0" rpy="0 0 0"/>
         <geometry>
-          <mesh filename="package://meshes/stl/iiwa_link_2.stl"/>
-        </geometry>
-        <material name="Orange"/>
-      </visual>
-      <collision>
-        <origin xyz="0 0 0" rpy="0 0 0"/>
-        <geometry>
-          <mesh filename="package://meshes/stl/iiwa_link_2.stl"/>
+          <mesh filename="package://meshes/stl/iiwa_link_2.stl" scale="0.001 0.001 0.001"/>
+        </geometry>
+        <material name="Orange"/>
+      </visual>
+      <collision>
+        <origin xyz="0 0 0" rpy="0 0 0"/>
+        <geometry>
+          <mesh filename="package://meshes/stl/iiwa_link_2.stl" scale="0.001 0.001 0.001"/>
         </geometry>
         <material name="Orange"/>
@@ -139,12 +140,12 @@
         <origin xyz="0 0 0" rpy="0 0 0"/>
         <geometry>
-          <mesh filename="package://meshes/stl/iiwa_link_3.stl"/>
-        </geometry>
-        <material name="Orange"/>
-      </visual>
-      <collision>
-        <origin xyz="0 0 0" rpy="0 0 0"/>
-        <geometry>
-          <mesh filename="package://meshes/stl/iiwa_link_3.stl"/>
+          <mesh filename="package://meshes/stl/iiwa_link_3.stl" scale="0.001 0.001 0.001"/>
+        </geometry>
+        <material name="Orange"/>
+      </visual>
+      <collision>
+        <origin xyz="0 0 0" rpy="0 0 0"/>
+        <geometry>
+          <mesh filename="package://meshes/stl/iiwa_link_3.stl" scale="0.001 0.001 0.001"/>
         </geometry>
         <material name="Orange"/>
@@ -174,12 +175,12 @@
         <origin xyz="0 0 0" rpy="0 0 0"/>
         <geometry>
-          <mesh filename="package://meshes/stl/iiwa_link_4.stl"/>
-        </geometry>
-        <material name="Orange"/>
-      </visual>
-      <collision>
-        <origin xyz="0 0 0" rpy="0 0 0"/>
-        <geometry>
-          <mesh filename="package://meshes/stl/iiwa_link_4.stl"/>
+          <mesh filename="package://meshes/stl/iiwa_link_4.stl" scale="0.001 0.001 0.001"/>
+        </geometry>
+        <material name="Orange"/>
+      </visual>
+      <collision>
+        <origin xyz="0 0 0" rpy="0 0 0"/>
+        <geometry>
+          <mesh filename="package://meshes/stl/iiwa_link_4.stl" scale="0.001 0.001 0.001"/>
         </geometry>
         <material name="Orange"/>
@@ -209,12 +210,12 @@
         <origin xyz="0 0 0" rpy="0 0 0"/>
         <geometry>
-          <mesh filename="package://meshes/stl/iiwa_link_5.stl"/>
-        </geometry>
-        <material name="Orange"/>
-      </visual>
-      <collision>
-        <origin xyz="0 0 0" rpy="0 0 0"/>
-        <geometry>
-          <mesh filename="package://meshes/stl/iiwa_link_5.stl"/>
+          <mesh filename="package://meshes/stl/iiwa_link_5.stl" scale="0.001 0.001 0.001"/>
+        </geometry>
+        <material name="Orange"/>
+      </visual>
+      <collision>
+        <origin xyz="0 0 0" rpy="0 0 0"/>
+        <geometry>
+          <mesh filename="package://meshes/stl/iiwa_link_5.stl" scale="0.001 0.001 0.001"/>
         </geometry>
         <material name="Orange"/>
@@ -244,12 +245,12 @@
         <origin xyz="0 0 0" rpy="0 0 0"/>
         <geometry>
-          <mesh filename="package://meshes/stl/iiwa_link_6.stl"/>
-        </geometry>
-        <material name="Orange"/>
-      </visual>
-      <collision>
-        <origin xyz="0 0 0" rpy="0 0 0"/>
-        <geometry>
-          <mesh filename="package://meshes/stl/iiwa_link_6.stl"/>
+          <mesh filename="package://meshes/stl/iiwa_link_6.stl" scale="0.001 0.001 0.001"/>
+        </geometry>
+        <material name="Orange"/>
+      </visual>
+      <collision>
+        <origin xyz="0 0 0" rpy="0 0 0"/>
+        <geometry>
+          <mesh filename="package://meshes/stl/iiwa_link_6.stl" scale="0.001 0.001 0.001"/>
         </geometry>
         <material name="Orange"/>
@@ -279,5 +280,5 @@
         <origin xyz="0 0 0" rpy="0 0 0"/>
         <geometry>
-          <mesh filename="package://meshes/stl/iiwa_link_7.stl"/>
+          <mesh filename="package://meshes/stl/iiwa_link_7.stl" scale="0.001 0.001 0.001"/>
         </geometry>
         <material name="Grey"/>
@@ -286,5 +287,5 @@
         <origin xyz="0 0 0" rpy="0 0 0"/>
         <geometry>
-          <mesh filename="package://meshes/stl/iiwa_link_7.stl"/>
+          <mesh filename="package://meshes/stl/iiwa_link_7.stl" scale="0.001 0.001 0.001"/>
         </geometry>
         <material name="Grey"/>
@@ -334,6 +335,6 @@
   </link>
     <!--Extensions -->
-    <xacro:iiwa_gazebo robot_name="KUKAiiwa14" />
-    <xacro:iiwa_transmission hardware_interface="${hardware_interface}"/>
+    <!-- <xacro:iiwa_gazebo robot_name="KUKAiiwa14" /> -->
+    <!-- <xacro:iiwa_transmission hardware_interface="${hardware_interface}"/> -->
   </xacro:macro>
 </robot>

Commit message: unsolved scaling problem with xacro -> urdf conversion

File: src/robot_properties_kuka/resources/pre_generated_urdf/iiwa.urdf (robot description, URDF)
Before this commit: robot KUKAiiwa, 9 links, 8 joints
Links:
- link contact: geometry visual mesh filename=package://meshes/sphere.obj scale=0.065 0.065 0.065
Joints:
- joint A2: limit effort=30 velocity=1.0 -> lower=-2.0944 upper=2.0944 effort=320 velocity=1.48353
- joint A3: limit effort=30 velocity=1.0 -> lower=-2.96706 upper=2.96706 effort=176 velocity=1.74533
- joint A4: limit effort=30 velocity=1.0 -> lower=-2.0944 upper=2.0944 effort=176 velocity=1.309
- joint A5: limit effort=30 velocity=1.0 -> lower=-2.96706 upper=2.96706 effort=110 velocity=2.26893
- joint A6: limit effort=30 velocity=1.0 -> lower=-2.0944 upper=2.0944 effort=40 velocity=2.35619
- joint A7: limit effort=30 velocity=1.0 -> lower=-3.05433 upper=3.05433 effort=40 velocity=2.35619

File: src/robot_properties_kuka/resources/xacro/iiwa.urdf.xacro (robot description, xacro)
@@ -2,13 +2,14 @@
 <robot name="KUKAiiwa14" xmlns:xacro="http://www.ros.org/wiki/xacro">
   <!-- Import Rviz colors -->
-  <xacro:include filename="materials.xacro" />
+  <!-- <xacro:include filename="materials.xacro" /> -->
   <!--Import the lbr iiwa macro -->
   <xacro:include filename="iiwa.xacro"/>
   <!-- Fix to world just for testing -->
-  <!-- <link name="world"/> -->
+  <link name="world"/>
   <!--KUKAiiwa14-->
+  <!-- <xacro:KUKAiiwa14 robot_name="KUKAiiwa14"/> -->
   <xacro:KUKAiiwa14 hardware_interface="PositionJointInterface" robot_name="KUKAiiwa14" parent="world">
   <!-- <xacro:KUKAiiwa14 parent="world"> -->
-    <origin xyz="0 0 0" rpy="0 0 0" />
-  </xacro:KUKAiiwa14>
+    <!-- <origin xyz="0 0 0" rpy="0 0 0" /> -->
+  <!-- </xacro:KUKAiiwa14> -->
 </robot>
