Commit message: fixed xacro problem

File: src/robot_properties_kuka/resources/xacro/iiwa.urdf.xacro (robot description, xacro)
@@ -2,5 +2,5 @@
 <robot name="KUKAiiwa14" xmlns:xacro="http://www.ros.org/wiki/xacro">
   <!-- Import Rviz colors -->
-  <!-- <xacro:include filename="materials.xacro" /> -->
+  <xacro:include filename="materials.xacro" />
   <!--Import the lbr iiwa macro -->
   <xacro:include filename="iiwa.xacro"/>
@@ -8,8 +8,8 @@
   <link name="world"/>
   <!--KUKAiiwa14-->
-  <!-- <xacro:KUKAiiwa14 robot_name="KUKAiiwa14"/> -->
-  <xacro:KUKAiiwa14 hardware_interface="PositionJointInterface" robot_name="KUKAiiwa14" parent="world">
+  <xacro:KUKAiiwa14 robot_name="KUKAiiwa14">
+  <!-- <xacro:KUKAiiwa14 hardware_interface="PositionJointInterface" robot_name="KUKAiiwa14" parent="world"> -->
   <!-- <xacro:KUKAiiwa14 parent="world"> -->
-    <!-- <origin xyz="0 0 0" rpy="0 0 0" /> -->
-  <!-- </xacro:KUKAiiwa14> -->
+    <origin xyz="0 0 0" rpy="0 0 0" />
+  </xacro:KUKAiiwa14>
 </robot>

File: src/robot_properties_kuka/resources/xacro/iiwa.xacro (robot description, xacro)
@@ -7,5 +7,4 @@
   <!-- Include Utilities -->
   <!-- <xacro:include filename="utilities.xacro" /> -->
-  <!-- <xacro:include filename="materials.xacro" /> -->
   <!-- some constants -->
   <xacro:property name="safety_controller_k_pos" value="100" />
@@ -14,41 +13,36 @@
   <xacro:macro name="KUKAiiwa14" params="robot_name *origin">
     <!--joint between WORLD and BASE-->
-    <!-- <joint name="A0" type="fixed">
+    <joint name="A0" type="fixed">
       <xacro:insert_block name="origin"/>
       <parent link="world"/>
       <child link="iiwa_base"/>
-    </joint> -->
+    </joint>
     <!-- BASE -->
     <link name="iiwa_base">
       <inertial>
-        <origin xyz="0.00000 0.00000 0.00000"/>
-        <mass value="8.00000"/>
-        <inertia ixx="0.00095" iyy="0.00133" izz="0.00118" ixy="0.00000" ixz="-0.00000" iyz="-0.00006"/>
-      </inertial>
-      <visual>
-        <origin xyz="0.0 0.0 0.0" rpy="0.0 0.0 0.0" />
-        <geometry>
-        <mesh>
-          <uri>package://meshes/stl/iiwa_base.stl</uri>
-          <scale>0.001 0.001 0.001</scale>
-        </mesh>
-        </geometry>
-        <!-- <material name="Grey"/> -->
-      </visual>
-      <collision>
-        <origin xyz="0 0 0" rpy="0 0 0"/>
-        <geometry>
-        <mesh>
-          <uri>package://meshes/stl/iiwa_base.stl</uri>
-          <scale>0.001 0.001 0.001</scale>
-        </mesh>        </geometry>
-        <!-- <material name="Grey"/> -->
-      </collision>
-      <!-- <self_collision_checking>
+        <origin xyz="0 0 0" rpy="0 0 0"/>
+        <mass value="5"/>
+        <inertia ixx="0.05"  ixy="0"  ixz="0" iyy="0.06" iyz="0" izz="0.03" />
+      </inertial>
+      <visual>
+        <origin xyz="0 0 0" rpy="0 0 0"/>
+        <geometry>
+          <mesh filename="package://meshes/stl/iiwa_base.stl" scale="0.001 0.001 0.001"/>
+        </geometry>
+        <material name="Grey"/>
+      </visual>
+      <collision>
+        <origin xyz="0 0 0" rpy="0 0 0"/>
+        <geometry>
+          <mesh filename="package://meshes/stl/iiwa_base.stl" scale="0.001 0.001 0.001"/>
+        </geometry>
+        <material name="Grey"/>
+      </collision>
+      <self_collision_checking>
         <origin xyz="0 0 0" rpy="0 0 0"/>
         <geometry>
           <capsule radius="0.15" length="0.25"/>
         </geometry>
-      </self_collision_checking> -->
+      </self_collision_checking>
     </link>
     <!-- joint between base and link1 -->
@@ -66,4 +60,281 @@
       <dynamics damping="${joint_damping}"/> -->
     </joint>
+    <!-- LINK 1-->
+    <link name="L1">
+      <inertial>
+        <origin xyz="0.00000 0.00000 0.00000"/>
+        <mass value="3.94781"/>
+        <inertia ixx="0.00455" iyy="0.00454" izz="0.00029" ixy="0.00000" ixz="-0.00000" iyz="-0.00001"/>
+      </inertial>
+      <visual>
+        <origin xyz="0 0 0" rpy="0 0 0"/>
+        <geometry>
+          <mesh filename="package://meshes/stl/iiwa_link_1.stl" scale="0.001 0.001 0.001"/>
+        </geometry>
+        <material name="Orange"/>
+      </visual>
+      <collision>
+        <origin xyz="0 0 0" rpy="0 0 0"/>
+        <geometry>
+          <mesh filename="package://meshes/stl/iiwa_link_1.stl" scale="0.001 0.001 0.001"/>
+        </geometry>
+        <material name="Orange"/>
+      </collision>
+    </link>
+    <!-- joint between link1 and link2 -->
+    <joint name="A2" type="revolute">
+      <origin xyz="0.00000 0.00000 0.20250" rpy="2.3561944901923457 -1.5707962635746238 2.3561944901923457"/>
+      <parent link="L1"/>
+      <child  link="L2"/>
+      <axis xyz="0 0 1"/>
+      <limit lower="-2.0944" upper="2.0944" velocity="1.48353" effort="320"/>
+      <!-- <safety_controller soft_lower_limit="${-118 * PI / 180}"
+                          soft_upper_limit="${118 * PI / 180}"
+                          k_position="${safety_controller_k_pos}"
+                          k_velocity="${safety_controller_k_vel}"/>
+      <dynamics damping="${joint_damping}"/> -->
+    </joint>
+    <!-- LINK 2-->
+    <link name="L2">
+      <inertial>
+        <origin xyz="0.0003 0.059 0.042" rpy="0 0 0"/>
+        <mass value="4"/>
+        <inertia ixx="0.05"  ixy="0"  ixz="0" iyy="0.018" iyz="0" izz="0.044" />
+      </inertial>
+      <visual>
+        <origin xyz="0 0 0" rpy="0 0 0"/>
+        <geometry>
+          <mesh filename="package://meshes/stl/iiwa_link_2.stl" scale="0.001 0.001 0.001"/>
+        </geometry>
+        <material name="Orange"/>
+      </visual>
+      <collision>
+        <origin xyz="0 0 0" rpy="0 0 0"/>
+        <geometry>
+          <mesh filename="package://meshes/stl/iiwa_link_2.stl" scale="0.001 0.001 0.001"/>
+        </geometry>
+        <material name="Orange"/>
+      </collision>
+    </link>
+    <!-- joint between link2 and link3 -->
+    <joint name="A3" type="revolute">
+      <origin xyz="0.20450 0.00000 0.00000" rpy="1.5707963267948948 -4.371139000186238E-8 1.5707963705062866"/>
+      <parent link="L2"/>
+      <child  link="L3"/>
+      <axis xyz="0 0 1"/>
+      <limit lower="-2.96706" upper="2.96706" velocity="1.74533" effort="176"/>
+      <!-- <safety_controller soft_lower_limit="${-168 * PI / 180}"
+                          soft_upper_limit="${168 * PI / 180}"
+                          k_position="${safety_controller_k_pos}"
+                          k_velocity="${safety_controller_k_vel}"/>
+      <dynamics damping="${joint_damping}"/> -->
+    </joint>
+    <!-- LINK 3-->
+    <link name="L3">
+      <inertial>
+        <origin xyz="0 0.03 0.13" rpy="0 0 0"/>
+        <mass value="3"/>
+        <inertia ixx="0.08"  ixy="0"  ixz="0" iyy="0.075" iyz="0" izz="0.01" />
+      </inertial>
+      <visual>
+        <origin xyz="0 0 0" rpy="0 0 0"/>
+        <geometry>
+          <mesh filename="package://meshes/stl/iiwa_link_3.stl" scale="0.001 0.001 0.001"/>
+        </geometry>
+        <material name="Orange"/>
+      </visual>
+      <collision>
+        <origin xyz="0 0 0" rpy="0 0 0"/>
+        <geometry>
+          <mesh filename="package://meshes/stl/iiwa_link_3.stl" scale="0.001 0.001 0.001"/>
+        </geometry>
+        <material name="Orange"/>
+      </collision>
+    </link>
+    <!-- joint between link3 and link4 -->
+    <joint name="A4" type="revolute">
+      <origin xyz="0.00000 0.00000 0.21550" rpy="1.5707963705062866 -0.0 0.0"/>
+      <parent link="L3"/>
+      <child  link="L4"/>
+      <axis xyz="0 0 1"/>
+      <limit lower="-2.0944" upper="2.0944" velocity="1.309" effort="176"/>
+      <!-- <safety_controller soft_lower_limit="${-118 * PI / 180}"
+                          soft_upper_limit="${118 * PI / 180}"
+                          k_position="${safety_controller_k_pos}"
+                          k_velocity="${safety_controller_k_vel}"/>
+      <dynamics damping="${joint_damping}"/> -->
+    </joint>
+    <!-- LINK 4-->
+    <link name="L4">
+      <inertial>
+        <origin xyz="0 0.067 0.034" rpy="0 0 0"/>
+        <mass value="2.7"/>
+        <inertia ixx="0.03"  ixy="0"  ixz="0" iyy="0.01" iyz="0" izz="0.029" />
+      </inertial>
+      <visual>
+        <origin xyz="0 0 0" rpy="0 0 0"/>
+        <geometry>
+          <mesh filename="package://meshes/stl/iiwa_link_4.stl" scale="0.001 0.001 0.001"/>
+        </geometry>
+        <material name="Orange"/>
+      </visual>
+      <collision>
+        <origin xyz="0 0 0" rpy="0 0 0"/>
+        <geometry>
+          <mesh filename="package://meshes/stl/iiwa_link_4.stl" scale="0.001 0.001 0.001"/>
+        </geometry>
+        <material name="Orange"/>
+      </collision>
+    </link>
+    <!-- joint between link4 and link5 -->
+    <joint name="A5" type="revolute">
+      <origin xyz="0.00000 0.18450 0.00000" rpy="-1.5707963705062866 0.0 -0.0"/>
+      <parent link="L4"/>
+      <child  link="L5"/>
+      <axis xyz="0 0 1"/>
+      <limit lower="-2.96706" upper="2.96706" velocity="2.26893" effort="110"/>
+      <!-- <safety_controller soft_lower_limit="${-168 * PI / 180}"
+                          soft_upper_limit="${168 * PI / 180}"
+                          k_position="${safety_controller_k_pos}"
+                          k_velocity="${safety_controller_k_vel}"/>
+      <dynamics damping="${joint_damping}"/> -->
+    </joint>
+    <!-- LINK 5-->
+    <link name="L5">
+      <inertial>
+        <origin xyz="0.0001 0.021 0.076" rpy="0 0 0"/>
+        <mass value="1.7"/>
+        <inertia ixx="0.02"  ixy="0"  ixz="0" iyy="0.018" iyz="0" izz="0.005" />
+      </inertial>
+      <visual>
+        <origin xyz="0 0 0" rpy="0 0 0"/>
+        <geometry>
+          <mesh filename="package://meshes/stl/iiwa_link_5.stl" scale="0.001 0.001 0.001"/>
+        </geometry>
+        <material name="Orange"/>
+      </visual>
+      <collision>
+        <origin xyz="0 0 0" rpy="0 0 0"/>
+        <geometry>
+          <mesh filename="package://meshes/stl/iiwa_link_5.stl" scale="0.001 0.001 0.001"/>
+        </geometry>
+        <material name="Orange"/>
+      </collision>
+    </link>
+    <!-- joint between link5 and link6 -->
+    <joint name="A6" type="revolute">
+      <origin xyz="0.00000 -0.06070 0.21550" rpy="2.3561944901923457 -1.5707962635746238 2.3561944901923457"/>
+      <parent link="L5"/>
+      <child  link="L6"/>
+      <axis xyz="0 0 1"/>
+      <limit lower="-2.0944" upper="2.0944" velocity="2.35619" effort="40"/>
+      <!-- <safety_controller soft_lower_limit="${-118 * PI / 180}"
+                          soft_upper_limit="${118 * PI / 180}"
+                          k_position="${safety_controller_k_pos}"
+                          k_velocity="${safety_controller_k_vel}"/>
+      <dynamics damping="${joint_damping}"/> -->
+    </joint>
+    <!-- LINK 6-->
+    <link name="L6">
+      <inertial>
+        <origin xyz="0 0.0006 0.0004" rpy="0 0 0"/>
+        <mass value="1.8"/>
+        <inertia ixx="0.005"  ixy="0"  ixz="0" iyy="0.0036" iyz="0" izz="0.0047" />
+      </inertial>
+      <visual>
+        <origin xyz="0 0 0" rpy="0 0 0"/>
+        <geometry>
+          <mesh filename="package://meshes/stl/iiwa_link_6.stl" scale="0.001 0.001 0.001"/>
+        </geometry>
+        <material name="Orange"/>
+      </visual>
+      <collision>
+        <origin xyz="0 0 0" rpy="0 0 0"/>
+        <geometry>
+          <mesh filename="package://meshes/stl/iiwa_link_6.stl" scale="0.001 0.001 0.001"/>
+        </geometry>
+        <material name="Orange"/>
+      </collision>
+    </link>
+    <!-- joint between link6 and link7 -->
+    <joint name="A7" type="revolute">
+      <origin xyz="0.08100 0.00000 0.06070" rpy="1.5707963267948948 -4.371139000186238E-8 1.5707963705062866"/>
+      <parent link="L6"/>
+      <child  link="L7"/>
+      <axis xyz="0 0 1"/>
+      <limit lower="-3.05433" upper="3.05433" velocity="2.35619" effort="40" />
+      <!-- <safety_controller soft_lower_limit="${-173 * PI / 180}"
+                          soft_upper_limit="${173 * PI / 180}"
+                          k_position="${safety_controller_k_pos}"
+                          k_velocity="${safety_controller_k_vel}"/>
+      <dynamics damping="${joint_damping}"/> -->
+    </joint>
+    <!-- LINK 7-->
+    <link name="L7">
+      <inertial>
+        <origin xyz="0 0 0.02" rpy="0 0 0"/>
+        <mass value="0.3"/>
+        <inertia ixx="0.001"  ixy="0"  ixz="0" iyy="0.001" iyz="0" izz="0.001" />
+      </inertial>
+      <visual>
+        <origin xyz="0 0 0" rpy="0 0 0"/>
+        <geometry>
+          <mesh filename="package://meshes/stl/iiwa_link_7.stl" scale="0.001 0.001 0.001"/>
+        </geometry>
+        <material name="Grey"/>
+      </visual>
+      <collision>
+        <origin xyz="0 0 0" rpy="0 0 0"/>
+        <geometry>
+          <mesh filename="package://meshes/stl/iiwa_link_7.stl" scale="0.001 0.001 0.001"/>
+        </geometry>
+        <material name="Grey"/>
+      </collision>
+    </link>
+    <!-- EE -->
+    <joint name="EE" type="fixed">
+      <parent link="L7"/>
+      <child link="contact"/>
+      <!-- Joint placement -->
+      <origin rpy="0 0 0" xyz="0 0.0 0.04"/>
+      <!-- Limits (usefull?) -->
+      <limit effort="1000" lower="-10" upper="10" velocity="1000"/>
+      <!-- pybullet simulation parameters -->
+      <dynamics damping="0.0" friction="0.0"/>
+    </joint>
+    <!-- CONTACT (modeled by a tennis ball) -->
+    <link name="contact">
+      <inertial>
+        <origin rpy="0 0 0" xyz="0 0 0.0"/>
+        <mass value="0.057"/>
+        <inertia ixx="0.0000354" ixy="0.0" ixz="0.0" iyy="0.0000354" iyz="0.0" izz="0.0000354"/>
+      </inertial>
+      <visual>
+        <origin rpy="0 0 0" xyz="0 0 0"/>
+        <geometry>
+          <mesh filename="package://meshes/sphere.obj" scale="0.065 0.065 0.065"/>/>
+        </geometry>
+        <material name="grey">
+          <color rgba="0.8 0.8 0.8 1.0"/>
+        </material>
+      </visual>
+      <collision>
+        <origin rpy="0 0 0" xyz="0 0 0"/>
+        <geometry>
+          <mesh filename="package://meshes/sphere.obj" scale="0.065 0.065 0.065"/>/>
+        </geometry>
+        <material name="grey">
+          <color rgba="0.8 0.8 0.8 1.0"/>
+        </material>
+      </collision>
+      <!-- Bullet specific paramters -->
+      <contact>
+        <lateral_friction value="1.0"/>
+        <restitution value="0.5"/>
+      </contact>
+    </link>
+    <!--Extensions -->
+    <!-- <xacro:iiwa_gazebo robot_name="KUKAiiwa14" /> -->
+    <!-- <xacro:iiwa_transmission hardware_interface="${hardware_interface}"/> -->
   </xacro:macro>
 </robot>

Commit message: added transmission models in xacro + gazebo elements

File: src/robot_properties_kuka/resources/xacro/iiwa.urdf.xacro (robot description, xacro)
@@ -8,7 +8,5 @@
   <link name="world"/>
   <!--KUKAiiwa14-->
-  <xacro:KUKAiiwa14 robot_name="KUKAiiwa14">
-  <!-- <xacro:KUKAiiwa14 hardware_interface="PositionJointInterface" robot_name="KUKAiiwa14" parent="world"> -->
-  <!-- <xacro:KUKAiiwa14 parent="world"> -->
+  <xacro:KUKAiiwa14 robot_name="KUKAiiwa14" hardware_interface="PositionJointInterface">
     <origin xyz="0 0 0" rpy="0 0 0" />
   </xacro:KUKAiiwa14>

File: src/robot_properties_kuka/resources/xacro/iiwa.xacro (robot description, xacro)
@@ -2,9 +2,7 @@
 <robot xmlns:xacro="http://www.ros.org/wiki/xacro">
   <!-- Import all Gazebo-customization elements, including Gazebo colors -->
-  <!-- <xacro:include filename="iiwa.gazebo.xacro" /> -->
+  <xacro:include filename="iiwa.gazebo.xacro" />
   <!-- Import Transmissions -->
-  <!-- <xacro:include filename="iiwa.transmission.xacro" /> -->
-  <!-- Include Utilities -->
-  <!-- <xacro:include filename="utilities.xacro" /> -->
+  <xacro:include filename="iiwa.transmission.xacro" />
   <!-- some constants -->
   <xacro:property name="safety_controller_k_pos" value="100" />
@@ -54,9 +52,9 @@
       <axis xyz="0 0 1"/>
       <limit lower="-2.96706" upper="2.96706" velocity="1.48353" effort="320"/>
-      <!-- <safety_controller soft_lower_limit="${-168 * PI / 180}"
+      <safety_controller soft_lower_limit="${-168 * PI / 180}"
                           soft_upper_limit="${168 * PI / 180}"
                           k_position="${safety_controller_k_pos}"
                           k_velocity="${safety_controller_k_vel}"/>
-      <dynamics damping="${joint_damping}"/> -->
+      <dynamics damping="${joint_damping}"/>
     </joint>
     <!-- LINK 1-->
@@ -89,9 +87,9 @@
       <axis xyz="0 0 1"/>
       <limit lower="-2.0944" upper="2.0944" velocity="1.48353" effort="320"/>
-      <!-- <safety_controller soft_lower_limit="${-118 * PI / 180}"
+      <safety_controller soft_lower_limit="${-118 * PI / 180}"
                           soft_upper_limit="${118 * PI / 180}"
                           k_position="${safety_controller_k_pos}"
                           k_velocity="${safety_controller_k_vel}"/>
-      <dynamics damping="${joint_damping}"/> -->
+      <dynamics damping="${joint_damping}"/>
     </joint>
     <!-- LINK 2-->
@@ -124,9 +122,9 @@
       <axis xyz="0 0 1"/>
       <limit lower="-2.96706" upper="2.96706" velocity="1.74533" effort="176"/>
-      <!-- <safety_controller soft_lower_limit="${-168 * PI / 180}"
+      <safety_controller soft_lower_limit="${-168 * PI / 180}"
                           soft_upper_limit="${168 * PI / 180}"
                           k_position="${safety_controller_k_pos}"
                           k_velocity="${safety_controller_k_vel}"/>
-      <dynamics damping="${joint_damping}"/> -->
+      <dynamics damping="${joint_damping}"/>
     </joint>
     <!-- LINK 3-->
@@ -159,9 +157,9 @@
       <axis xyz="0 0 1"/>
       <limit lower="-2.0944" upper="2.0944" velocity="1.309" effort="176"/>
-      <!-- <safety_controller soft_lower_limit="${-118 * PI / 180}"
+      <safety_controller soft_lower_limit="${-118 * PI / 180}"
                           soft_upper_limit="${118 * PI / 180}"
                           k_position="${safety_controller_k_pos}"
                           k_velocity="${safety_controller_k_vel}"/>
-      <dynamics damping="${joint_damping}"/> -->
+      <dynamics damping="${joint_damping}"/>
     </joint>
     <!-- LINK 4-->
@@ -194,9 +192,9 @@
       <axis xyz="0 0 1"/>
       <limit lower="-2.96706" upper="2.96706" velocity="2.26893" effort="110"/>
-      <!-- <safety_controller soft_lower_limit="${-168 * PI / 180}"
+      <safety_controller soft_lower_limit="${-168 * PI / 180}"
                           soft_upper_limit="${168 * PI / 180}"
                           k_position="${safety_controller_k_pos}"
                           k_velocity="${safety_controller_k_vel}"/>
-      <dynamics damping="${joint_damping}"/> -->
+      <dynamics damping="${joint_damping}"/>
     </joint>
     <!-- LINK 5-->
@@ -229,9 +227,9 @@
       <axis xyz="0 0 1"/>
       <limit lower="-2.0944" upper="2.0944" velocity="2.35619" effort="40"/>
-      <!-- <safety_controller soft_lower_limit="${-118 * PI / 180}"
+      <safety_controller soft_lower_limit="${-118 * PI / 180}"
                           soft_upper_limit="${118 * PI / 180}"
                           k_position="${safety_controller_k_pos}"
                           k_velocity="${safety_controller_k_vel}"/>
-      <dynamics damping="${joint_damping}"/> -->
+      <dynamics damping="${joint_damping}"/>
     </joint>
     <!-- LINK 6-->
@@ -264,9 +262,9 @@
       <axis xyz="0 0 1"/>
       <limit lower="-3.05433" upper="3.05433" velocity="2.35619" effort="40" />
-      <!-- <safety_controller soft_lower_limit="${-173 * PI / 180}"
+      <safety_controller soft_lower_limit="${-173 * PI / 180}"
                           soft_upper_limit="${173 * PI / 180}"
                           k_position="${safety_controller_k_pos}"
                           k_velocity="${safety_controller_k_vel}"/>
-      <dynamics damping="${joint_damping}"/> -->
+      <dynamics damping="${joint_damping}"/>
     </joint>
     <!-- LINK 7-->
@@ -335,6 +333,6 @@
     </link>
     <!--Extensions -->
-    <!-- <xacro:iiwa_gazebo robot_name="KUKAiiwa14" /> -->
-    <!-- <xacro:iiwa_transmission hardware_interface="${hardware_interface}"/> -->
+    <xacro:iiwa_gazebo robot_name="KUKAiiwa14"/>
+    <xacro:iiwa_transmission hardware_interface="${hardware_interface}"/>
   </xacro:macro>
 </robot>
