Commit message: removed hw interface and soft limits bc bug

File: src/robot_properties_kuka/resources/xacro/iiwa.urdf.xacro (robot description, xacro)
@@ -8,5 +8,5 @@
   <link name="world"/>
   <!--KUKAiiwa14-->
-  <xacro:KUKAiiwa14 robot_name="KUKAiiwa14" hardware_interface="PositionJointInterface">
+  <xacro:KUKAiiwa14 robot_name="KUKAiiwa14"> <!-- hardware_interface="PositionJointInterface"> -->
     <origin xyz="0 0 0" rpy="0 0 0" />
   </xacro:KUKAiiwa14>

File: src/robot_properties_kuka/resources/xacro/iiwa.xacro (robot description, xacro)
@@ -52,9 +52,9 @@
       <axis xyz="0 0 1"/>
       <limit lower="-2.96706" upper="2.96706" velocity="1.48353" effort="320"/>
-      <safety_controller soft_lower_limit="${-168 * PI / 180}"
+      <!-- <safety_controller soft_lower_limit="${-168 * PI / 180}"
                           soft_upper_limit="${168 * PI / 180}"
                           k_position="${safety_controller_k_pos}"
                           k_velocity="${safety_controller_k_vel}"/>
-      <dynamics damping="${joint_damping}"/>
+      <dynamics damping="${joint_damping}"/> -->
     </joint>
     <!-- LINK 1-->
@@ -87,9 +87,9 @@
       <axis xyz="0 0 1"/>
       <limit lower="-2.0944" upper="2.0944" velocity="1.48353" effort="320"/>
-      <safety_controller soft_lower_limit="${-118 * PI / 180}"
+      <!-- <safety_controller soft_lower_limit="${-118 * PI / 180}"
                           soft_upper_limit="${118 * PI / 180}"
                           k_position="${safety_controller_k_pos}"
                           k_velocity="${safety_controller_k_vel}"/>
-      <dynamics damping="${joint_damping}"/>
+      <dynamics damping="${joint_damping}"/> -->
     </joint>
     <!-- LINK 2-->
@@ -122,9 +122,9 @@
       <axis xyz="0 0 1"/>
       <limit lower="-2.96706" upper="2.96706" velocity="1.74533" effort="176"/>
-      <safety_controller soft_lower_limit="${-168 * PI / 180}"
+      <!-- <safety_controller soft_lower_limit="${-168 * PI / 180}"
                           soft_upper_limit="${168 * PI / 180}"
                           k_position="${safety_controller_k_pos}"
                           k_velocity="${safety_controller_k_vel}"/>
-      <dynamics damping="${joint_damping}"/>
+      <dynamics damping="${joint_damping}"/> -->
     </joint>
     <!-- LINK 3-->
@@ -157,9 +157,9 @@
       <axis xyz="0 0 1"/>
       <limit lower="-2.0944" upper="2.0944" velocity="1.309" effort="176"/>
-      <safety_controller soft_lower_limit="${-118 * PI / 180}"
+      <!-- <safety_controller soft_lower_limit="${-118 * PI / 180}"
                           soft_upper_limit="${118 * PI / 180}"
                           k_position="${safety_controller_k_pos}"
                           k_velocity="${safety_controller_k_vel}"/>
-      <dynamics damping="${joint_damping}"/>
+      <dynamics damping="${joint_damping}"/> -->
     </joint>
     <!-- LINK 4-->
@@ -192,9 +192,9 @@
       <axis xyz="0 0 1"/>
       <limit lower="-2.96706" upper="2.96706" velocity="2.26893" effort="110"/>
-      <safety_controller soft_lower_limit="${-168 * PI / 180}"
+      <!-- <safety_controller soft_lower_limit="${-168 * PI / 180}"
                           soft_upper_limit="${168 * PI / 180}"
                           k_position="${safety_controller_k_pos}"
                           k_velocity="${safety_controller_k_vel}"/>
-      <dynamics damping="${joint_damping}"/>
+      <dynamics damping="${joint_damping}"/> -->
     </joint>
     <!-- LINK 5-->
@@ -227,9 +227,9 @@
       <axis xyz="0 0 1"/>
       <limit lower="-2.0944" upper="2.0944" velocity="2.35619" effort="40"/>
-      <safety_controller soft_lower_limit="${-118 * PI / 180}"
+      <!-- <safety_controller soft_lower_limit="${-118 * PI / 180}"
                           soft_upper_limit="${118 * PI / 180}"
                           k_position="${safety_controller_k_pos}"
                           k_velocity="${safety_controller_k_vel}"/>
-      <dynamics damping="${joint_damping}"/>
+      <dynamics damping="${joint_damping}"/> -->
     </joint>
     <!-- LINK 6-->
@@ -262,9 +262,9 @@
       <axis xyz="0 0 1"/>
       <limit lower="-3.05433" upper="3.05433" velocity="2.35619" effort="40" />
-      <safety_controller soft_lower_limit="${-173 * PI / 180}"
+      <!-- <safety_controller soft_lower_limit="${-173 * PI / 180}"
                           soft_upper_limit="${173 * PI / 180}"
                           k_position="${safety_controller_k_pos}"
                           k_velocity="${safety_controller_k_vel}"/>
-      <dynamics damping="${joint_damping}"/>
+      <dynamics damping="${joint_damping}"/> -->
     </joint>
     <!-- LINK 7-->
@@ -334,5 +334,5 @@
     <!--Extensions -->
     <xacro:iiwa_gazebo robot_name="KUKAiiwa14"/>
-    <xacro:iiwa_transmission hardware_interface="${hardware_interface}"/>
+    <!-- <xacro:iiwa_transmission hardware_interface="${hardware_interface}"/> -->
   </xacro:macro>
 </robot>
