Commit message: fails to integrate because pin robotwrapper and raisim have different ways of looking for meshes files

File: src/robot_properties_kuka/robot_properties_kuka/iiwa.urdf (robot description, URDF)
Before this commit: robot KUKAiiwa14, 10 links, 9 joints
Links:
- link L1: geometry collision mesh filename=package://robot_properties_kuka/meshes/iiwa_link_1.obj; visual mesh filename=package://robot_properties_kuka/meshes/iiwa_link_1.dae
- link L2: geometry collision mesh filename=package://robot_properties_kuka/meshes/iiwa_link_2.obj; visual mesh filename=package://robot_properties_kuka/meshes/iiwa_link_2.dae
- link L3: geometry collision mesh filename=package://robot_properties_kuka/meshes/iiwa_link_3.obj; visual mesh filename=package://robot_properties_kuka/meshes/iiwa_link_3.dae
- link L4: geometry collision mesh filename=package://robot_properties_kuka/meshes/iiwa_link_4.obj; visual mesh filename=package://robot_properties_kuka/meshes/iiwa_link_4.dae
- link L5: geometry collision mesh filename=package://robot_properties_kuka/meshes/iiwa_link_5.obj; visual mesh filename=package://robot_properties_kuka/meshes/iiwa_link_5.dae
- link L6: geometry collision mesh filename=package://robot_properties_kuka/meshes/iiwa_link_6.obj; visual mesh filename=package://robot_properties_kuka/meshes/iiwa_link_6.dae
- link L7: geometry collision mesh filename=package://robot_properties_kuka/meshes/iiwa_link_7.obj; visual mesh filename=package://robot_properties_kuka/meshes/iiwa_link_7.dae
- link iiwa_base: geometry collision mesh filename=package://robot_properties_kuka/meshes/iiwa_base.obj; visual mesh filename=package://robot_properties_kuka/meshes/iiwa_base.dae

File: src/robot_properties_kuka/robot_properties_kuka/xacro/iiwa.xacro (robot description, xacro)
@@ -26,5 +26,5 @@
         <origin xyz="0 0 0" rpy="0 0 0"/>
         <geometry>
-          <mesh filename="package://robot_properties_kuka/meshes/stl/iiwa_base.stl" />
+          <mesh filename="package://robot_properties_kuka/meshes/obj/iiwa_base.obj" />
         </geometry>
         <material name="Grey"/>
@@ -33,5 +33,5 @@
         <origin xyz="0 0 0" rpy="0 0 0"/>
         <geometry>
-          <mesh filename="package://robot_properties_kuka/meshes/stl/iiwa_base.stl" />
+          <mesh filename="package://robot_properties_kuka/meshes/obj/iiwa_base.obj" />
         </geometry>
         <material name="Grey"/>
@@ -67,12 +67,12 @@
         <origin xyz="0 0 0" rpy="0 0 0"/>
         <geometry>
-          <mesh filename="package://robot_properties_kuka/meshes/stl/iiwa_link_1.stl" />
-        </geometry>
-        <material name="Orange"/>
-      </visual>
-      <collision>
-        <origin xyz="0 0 0" rpy="0 0 0"/>
-        <geometry>
-          <mesh filename="package://robot_properties_kuka/meshes/stl/iiwa_link_1.stl" />
+          <mesh filename="package://robot_properties_kuka/meshes/obj/iiwa_link_1.obj" />
+        </geometry>
+        <material name="Orange"/>
+      </visual>
+      <collision>
+        <origin xyz="0 0 0" rpy="0 0 0"/>
+        <geometry>
+          <mesh filename="package://robot_properties_kuka/meshes/obj/iiwa_link_1.obj" />
         </geometry>
         <material name="Orange"/>
@@ -102,12 +102,12 @@
         <origin xyz="0 0 0" rpy="0 0 0"/>
         <geometry>
-          <mesh filename="package://robot_properties_kuka/meshes/stl/iiwa_link_2.stl" />
-        </geometry>
-        <material name="Orange"/>
-      </visual>
-      <collision>
-        <origin xyz="0 0 0" rpy="0 0 0"/>
-        <geometry>
-          <mesh filename="package://robot_properties_kuka/meshes/stl/iiwa_link_2.stl" />
+          <mesh filename="package://robot_properties_kuka/meshes/obj/iiwa_link_2.obj" />
+        </geometry>
+        <material name="Orange"/>
+      </visual>
+      <collision>
+        <origin xyz="0 0 0" rpy="0 0 0"/>
+        <geometry>
+          <mesh filename="package://robot_properties_kuka/meshes/obj/iiwa_link_2.obj" />
         </geometry>
         <material name="Orange"/>
@@ -137,12 +137,12 @@
         <origin xyz="0 0 0" rpy="0 0 0"/>
         <geometry>
-          <mesh filename="package://robot_properties_kuka/meshes/stl/iiwa_link_3.stl" />
-        </geometry>
-        <material name="Orange"/>
-      </visual>
-      <collision>
-        <origin xyz="0 0 0" rpy="0 0 0"/>
-        <geometry>
-          <mesh filename="package://robot_properties_kuka/meshes/stl/iiwa_link_3.stl" />
+          <mesh filename="package://robot_properties_kuka/meshes/obj/iiwa_link_3.obj" />
+        </geometry>
+        <material name="Orange"/>
+      </visual>
+      <collision>
+        <origin xyz="0 0 0" rpy="0 0 0"/>
+        <geometry>
+          <mesh filename="package://robot_properties_kuka/meshes/obj/iiwa_link_3.obj" />
         </geometry>
         <material name="Orange"/>
@@ -172,12 +172,12 @@
         <origin xyz="0 0 0" rpy="0 0 0"/>
         <geometry>
-          <mesh filename="package://robot_properties_kuka/meshes/stl/iiwa_link_4.stl" />
-        </geometry>
-        <material name="Orange"/>
-      </visual>
-      <collision>
-        <origin xyz="0 0 0" rpy="0 0 0"/>
-        <geometry>
-          <mesh filename="package://robot_properties_kuka/meshes/stl/iiwa_link_4.stl" />
+          <mesh filename="package://robot_properties_kuka/meshes/obj/iiwa_link_4.obj" />
+        </geometry>
+        <material name="Orange"/>
+      </visual>
+      <collision>
+        <origin xyz="0 0 0" rpy="0 0 0"/>
+        <geometry>
+          <mesh filename="package://robot_properties_kuka/meshes/obj/iiwa_link_4.obj" />
         </geometry>
         <material name="Orange"/>
@@ -207,12 +207,12 @@
         <origin xyz="0 0 0" rpy="0 0 0"/>
         <geometry>
-          <mesh filename="package://robot_properties_kuka/meshes/stl/iiwa_link_5.stl" />
-        </geometry>
-        <material name="Orange"/>
-      </visual>
-      <collision>
-        <origin xyz="0 0 0" rpy="0 0 0"/>
-        <geometry>
-          <mesh filename="package://robot_properties_kuka/meshes/stl/iiwa_link_5.stl" />
+          <mesh filename="package://robot_properties_kuka/meshes/obj/iiwa_link_5.obj" />
+        </geometry>
+        <material name="Orange"/>
+      </visual>
+      <collision>
+        <origin xyz="0 0 0" rpy="0 0 0"/>
+        <geometry>
+          <mesh filename="package://robot_properties_kuka/meshes/obj/iiwa_link_5.obj" />
         </geometry>
         <material name="Orange"/>
@@ -242,12 +242,12 @@
         <origin xyz="0 0 0" rpy="0 0 0"/>
         <geometry>
-          <mesh filename="package://robot_properties_kuka/meshes/stl/iiwa_link_6.stl" />
-        </geometry>
-        <material name="Orange"/>
-      </visual>
-      <collision>
-        <origin xyz="0 0 0" rpy="0 0 0"/>
-        <geometry>
-          <mesh filename="package://robot_properties_kuka/meshes/stl/iiwa_link_6.stl" />
+          <mesh filename="package://robot_properties_kuka/meshes/obj/iiwa_link_6.obj" />
+        </geometry>
+        <material name="Orange"/>
+      </visual>
+      <collision>
+        <origin xyz="0 0 0" rpy="0 0 0"/>
+        <geometry>
+          <mesh filename="package://robot_properties_kuka/meshes/obj/iiwa_link_6.obj" />
         </geometry>
         <material name="Orange"/>
@@ -277,5 +277,5 @@
         <origin xyz="0 0 0" rpy="0 0 0"/>
         <geometry>
-          <mesh filename="package://robot_properties_kuka/meshes/stl/iiwa_link_7.stl" />
+          <mesh filename="package://robot_properties_kuka/meshes/obj/iiwa_link_7.obj" />
         </geometry>
         <material name="Grey"/>
@@ -284,5 +284,5 @@
         <origin xyz="0 0 0" rpy="0 0 0"/>
         <geometry>
-          <mesh filename="package://robot_properties_kuka/meshes/stl/iiwa_link_7.stl" />
+          <mesh filename="package://robot_properties_kuka/meshes/obj/iiwa_link_7.obj" />
         </geometry>
         <material name="Grey"/>

Commit message: updated mass and inertia params based on sys ID paper. this improves gravity compensation accuracy

File: src/robot_properties_kuka/robot_properties_kuka/iiwa.urdf (robot description, URDF)
Before this commit: robot KUKAiiwa14, 10 links, 9 joints
Links:
- link L2: mass 4 -> 4.50275
- link L3: mass 3 -> 2.45520
- link L4: mass 2.7 -> 2.61155
- link L5: mass 1.7 -> 3.41000
- link L6: mass 1.8 -> 3.38795
- link L7: mass 0.3 -> 0.35432

File: src/robot_properties_kuka/robot_properties_kuka/xacro/iiwa.xacro (robot description, xacro)
@@ -96,6 +96,6 @@
       <inertial>
         <origin xyz="0.0003 0.059 0.042" rpy="0 0 0"/>
-        <mass value="4"/>
-        <inertia ixx="0.05"  ixy="0"  ixz="0" iyy="0.018" iyz="0" izz="0.044" />
+        <mass value="4.50275"/>
+        <inertia ixx="0.00032"  ixy="0"  ixz="0" iyy="0.00010" iyz="0" izz="0.00042" />
       </inertial>
       <visual>
@@ -131,6 +131,6 @@
       <inertial>
         <origin xyz="0 0.03 0.13" rpy="0 0 0"/>
-        <mass value="3"/>
-        <inertia ixx="0.08"  ixy="0"  ixz="0" iyy="0.075" iyz="0" izz="0.01" />
+        <mass value="2.45520"/>
+        <inertia ixx="0.00223"  ixy="-0.00005"  ixz="0.00007" iyy="0.00219" iyz="0.00007" izz="0.00073" />
       </inertial>
       <visual>
@@ -166,6 +166,6 @@
       <inertial>
         <origin xyz="0 0.067 0.034" rpy="0 0 0"/>
-        <mass value="2.7"/>
-        <inertia ixx="0.03"  ixy="0"  ixz="0" iyy="0.01" iyz="0" izz="0.029" />
+        <mass value="2.61155"/>
+        <inertia ixx="0.03844"  ixy="0.00088"  ixz="-0.00112" iyy="0.01144" iyz="-0.00111" izz="0.04988" />
       </inertial>
       <visual>
@@ -201,6 +201,6 @@
       <inertial>
         <origin xyz="0.0001 0.021 0.076" rpy="0 0 0"/>
-        <mass value="1.7"/>
-        <inertia ixx="0.02"  ixy="0"  ixz="0" iyy="0.018" iyz="0" izz="0.005" />
+        <mass value="3.41000"/>
+        <inertia ixx="0.00277"  ixy="-0.00001"  ixz="0.00001" iyy="0.00284" iyz="0" izz="0.00012" />
       </inertial>
       <visual>
@@ -236,6 +236,6 @@
       <inertial>
         <origin xyz="0 0.0006 0.0004" rpy="0 0 0"/>
-        <mass value="1.8"/>
-        <inertia ixx="0.005"  ixy="0"  ixz="0" iyy="0.0036" iyz="0" izz="0.0047" />
+        <mass value="3.38795"/>
+        <inertia ixx="0.00050"  ixy="-0.00005"  ixz="-0.00003" iyy="0.00281" iyz="-0.00004" izz="0.00232" />
       </inertial>
       <visual>
@@ -271,6 +271,6 @@
       <inertial>
         <origin xyz="0 0 0.02" rpy="0 0 0"/>
-        <mass value="0.3"/>
-        <inertia ixx="0.001"  ixy="0"  ixz="0" iyy="0.001" iyz="0" izz="0.001" />
+        <mass value="0.35432"/>
+        <inertia ixx="0.00795"  ixy="0.00022"  ixz="-0.00029" iyy="0.01089" iyz="-0.00029" izz="0.00294" />
       </inertial>
       <visual>
