Commit message: fixed meshes issue in robot wrapper

File: src/robot_properties_kuka/robot_properties_kuka/xacro/iiwa.xacro (robot description, xacro)
@@ -26,5 +26,5 @@
         <origin xyz="0 0 0" rpy="0 0 0"/>
         <geometry>
-          <mesh filename="package://meshes/stl/iiwa_base.stl" scale="0.001 0.001 0.001"/>
+          <mesh filename="package://robot_properties_kuka/meshes/stl/iiwa_base.stl" />
         </geometry>
         <material name="Grey"/>
@@ -33,5 +33,5 @@
         <origin xyz="0 0 0" rpy="0 0 0"/>
         <geometry>
-          <mesh filename="package://meshes/stl/iiwa_base.stl" scale="0.001 0.001 0.001"/>
+          <mesh filename="package://robot_properties_kuka/meshes/stl/iiwa_base.stl" />
         </geometry>
         <material name="Grey"/>
@@ -68,12 +68,12 @@
         <origin xyz="0 0 0" rpy="0 0 0"/>
         <geometry>
-          <mesh filename="package://meshes/stl/iiwa_link_1.stl" scale="0.001 0.001 0.001"/>
-        </geometry>
-        <material name="Orange"/>
-      </visual>
-      <collision>
-        <origin xyz="0 0 0" rpy="0 0 0"/>
-        <geometry>
-          <mesh filename="package://meshes/stl/iiwa_link_1.stl" scale="0.001 0.001 0.001"/>
+          <mesh filename="package://robot_properties_kuka/meshes/stl/iiwa_link_1.stl" />
+        </geometry>
+        <material name="Orange"/>
+      </visual>
+      <collision>
+        <origin xyz="0 0 0" rpy="0 0 0"/>
+        <geometry>
+          <mesh filename="package://robot_properties_kuka/meshes/stl/iiwa_link_1.stl" />
         </geometry>
         <material name="Orange"/>
@@ -103,12 +103,12 @@
         <origin xyz="0 0 0" rpy="0 0 0"/>
         <geometry>
-          <mesh filename="package://meshes/stl/iiwa_link_2.stl" scale="0.001 0.001 0.001"/>
-        </geometry>
-        <material name="Orange"/>
-      </visual>
-      <collision>
-        <origin xyz="0 0 0" rpy="0 0 0"/>
-        <geometry>
-          <mesh filename="package://meshes/stl/iiwa_link_2.stl" scale="0.001 0.001 0.001"/>
+          <mesh filename="package://robot_properties_kuka/meshes/stl/iiwa_link_2.stl" />
+        </geometry>
+        <material name="Orange"/>
+      </visual>
+      <collision>
+        <origin xyz="0 0 0" rpy="0 0 0"/>
+        <geometry>
+          <mesh filename="package://robot_properties_kuka/meshes/stl/iiwa_link_2.stl" />
         </geometry>
         <material name="Orange"/>
@@ -138,12 +138,12 @@
         <origin xyz="0 0 0" rpy="0 0 0"/>
         <geometry>
-          <mesh filename="package://meshes/stl/iiwa_link_3.stl" scale="0.001 0.001 0.001"/>
-        </geometry>
-        <material name="Orange"/>
-      </visual>
-      <collision>
-        <origin xyz="0 0 0" rpy="0 0 0"/>
-        <geometry>
-          <mesh filename="package://meshes/stl/iiwa_link_3.stl" scale="0.001 0.001 0.001"/>
+          <mesh filename="package://robot_properties_kuka/meshes/stl/iiwa_link_3.stl" />
+        </geometry>
+        <material name="Orange"/>
+      </visual>
+      <collision>
+        <origin xyz="0 0 0" rpy="0 0 0"/>
+        <geometry>
+          <mesh filename="package://robot_properties_kuka/meshes/stl/iiwa_link_3.stl" />
         </geometry>
         <material name="Orange"/>
@@ -173,12 +173,12 @@
         <origin xyz="0 0 0" rpy="0 0 0"/>
         <geometry>
-          <mesh filename="package://meshes/stl/iiwa_link_4.stl" scale="0.001 0.001 0.001"/>
-        </geometry>
-        <material name="Orange"/>
-      </visual>
-      <collision>
-        <origin xyz="0 0 0" rpy="0 0 0"/>
-        <geometry>
-          <mesh filename="package://meshes/stl/iiwa_link_4.stl" scale="0.001 0.001 0.001"/>
+          <mesh filename="package://robot_properties_kuka/meshes/stl/iiwa_link_4.stl" />
+        </geometry>
+        <material name="Orange"/>
+      </visual>
+      <collision>
+        <origin xyz="0 0 0" rpy="0 0 0"/>
+        <geometry>
+          <mesh filename="package://robot_properties_kuka/meshes/stl/iiwa_link_4.stl" />
         </geometry>
         <material name="Orange"/>
@@ -208,12 +208,12 @@
         <origin xyz="0 0 0" rpy="0 0 0"/>
         <geometry>
-          <mesh filename="package://meshes/stl/iiwa_link_5.stl" scale="0.001 0.001 0.001"/>
-        </geometry>
-        <material name="Orange"/>
-      </visual>
-      <collision>
-        <origin xyz="0 0 0" rpy="0 0 0"/>
-        <geometry>
-          <mesh filename="package://meshes/stl/iiwa_link_5.stl" scale="0.001 0.001 0.001"/>
+          <mesh filename="package://robot_properties_kuka/meshes/stl/iiwa_link_5.stl" />
+        </geometry>
+        <material name="Orange"/>
+      </visual>
+      <collision>
+        <origin xyz="0 0 0" rpy="0 0 0"/>
+        <geometry>
+          <mesh filename="package://robot_properties_kuka/meshes/stl/iiwa_link_5.stl" />
         </geometry>
         <material name="Orange"/>
@@ -243,12 +243,12 @@
         <origin xyz="0 0 0" rpy="0 0 0"/>
         <geometry>
-          <mesh filename="package://meshes/stl/iiwa_link_6.stl" scale="0.001 0.001 0.001"/>
-        </geometry>
-        <material name="Orange"/>
-      </visual>
-      <collision>
-        <origin xyz="0 0 0" rpy="0 0 0"/>
-        <geometry>
-          <mesh filename="package://meshes/stl/iiwa_link_6.stl" scale="0.001 0.001 0.001"/>
+          <mesh filename="package://robot_properties_kuka/meshes/stl/iiwa_link_6.stl" />
+        </geometry>
+        <material name="Orange"/>
+      </visual>
+      <collision>
+        <origin xyz="0 0 0" rpy="0 0 0"/>
+        <geometry>
+          <mesh filename="package://robot_properties_kuka/meshes/stl/iiwa_link_6.stl" />
         </geometry>
         <material name="Orange"/>
@@ -278,5 +278,5 @@
         <origin xyz="0 0 0" rpy="0 0 0"/>
         <geometry>
-          <mesh filename="package://meshes/stl/iiwa_link_7.stl" scale="0.001 0.001 0.001"/>
+          <mesh filename="package://robot_properties_kuka/meshes/stl/iiwa_link_7.stl" />
         </geometry>
         <material name="Grey"/>
@@ -285,5 +285,5 @@
         <origin xyz="0 0 0" rpy="0 0 0"/>
         <geometry>
-          <mesh filename="package://meshes/stl/iiwa_link_7.stl" scale="0.001 0.001 0.001"/>
+          <mesh filename="package://robot_properties_kuka/meshes/stl/iiwa_link_7.stl" />
         </geometry>
         <material name="Grey"/>
@@ -311,5 +311,5 @@
         <origin rpy="0 0 0" xyz="0 0 0"/>
         <geometry>
-          <mesh filename="package://meshes/sphere.obj" scale="0.065 0.065 0.065"/>/>
+          <mesh filename="package://robot_properties_kuka/meshes/sphere.obj" scale="0.065 0.065 0.065"/>/>
         </geometry>
         <material name="grey">
@@ -320,5 +320,5 @@
         <origin rpy="0 0 0" xyz="0 0 0"/>
         <geometry>
-          <mesh filename="package://meshes/sphere.obj" scale="0.065 0.065 0.065"/>/>
+          <mesh filename="package://robot_properties_kuka/meshes/sphere.obj" scale="0.065 0.065 0.065"/>/>
         </geometry>
         <material name="grey">

Commit message: resized manually stl and obj files to avoid the mesh rendering issue with large scales in osg

File: src/robot_properties_kuka/robot_properties_kuka/xacro/iiwa.xacro (robot description, xacro)
@@ -26,5 +26,5 @@
         <origin xyz="0 0 0" rpy="0 0 0"/>
         <geometry>
-          <mesh filename="package://robot_properties_kuka/meshes/stl/iiwa_base.stl" />
+          <mesh filename="package://robot_properties_kuka/meshes/stl/iiwa_base.dae" scale="0.001 0.001 0.001"/>
         </geometry>
         <material name="Grey"/>
@@ -33,5 +33,5 @@
         <origin xyz="0 0 0" rpy="0 0 0"/>
         <geometry>
-          <mesh filename="package://robot_properties_kuka/meshes/stl/iiwa_base.stl" />
+          <mesh filename="package://robot_properties_kuka/meshes/stl/iiwa_base.dae" scale="0.001 0.001 0.001"/>
         </geometry>
         <material name="Grey"/>
@@ -68,12 +68,12 @@
         <origin xyz="0 0 0" rpy="0 0 0"/>
         <geometry>
-          <mesh filename="package://robot_properties_kuka/meshes/stl/iiwa_link_1.stl" />
-        </geometry>
-        <material name="Orange"/>
-      </visual>
-      <collision>
-        <origin xyz="0 0 0" rpy="0 0 0"/>
-        <geometry>
-          <mesh filename="package://robot_properties_kuka/meshes/stl/iiwa_link_1.stl" />
+          <mesh filename="package://robot_properties_kuka/meshes/stl/iiwa_link_1.dae" scale="0.001 0.001 0.001"/>
+        </geometry>
+        <material name="Orange"/>
+      </visual>
+      <collision>
+        <origin xyz="0 0 0" rpy="0 0 0"/>
+        <geometry>
+          <mesh filename="package://robot_properties_kuka/meshes/stl/iiwa_link_1.dae" scale="0.001 0.001 0.001"/>
         </geometry>
         <material name="Orange"/>
@@ -103,12 +103,12 @@
         <origin xyz="0 0 0" rpy="0 0 0"/>
         <geometry>
-          <mesh filename="package://robot_properties_kuka/meshes/stl/iiwa_link_2.stl" />
-        </geometry>
-        <material name="Orange"/>
-      </visual>
-      <collision>
-        <origin xyz="0 0 0" rpy="0 0 0"/>
-        <geometry>
-          <mesh filename="package://robot_properties_kuka/meshes/stl/iiwa_link_2.stl" />
+          <mesh filename="package://robot_properties_kuka/meshes/stl/iiwa_link_2.dae" scale="0.001 0.001 0.001"/>
+        </geometry>
+        <material name="Orange"/>
+      </visual>
+      <collision>
+        <origin xyz="0 0 0" rpy="0 0 0"/>
+        <geometry>
+          <mesh filename="package://robot_properties_kuka/meshes/stl/iiwa_link_2.dae" scale="0.001 0.001 0.001"/>
         </geometry>
         <material name="Orange"/>
@@ -138,12 +138,12 @@
         <origin xyz="0 0 0" rpy="0 0 0"/>
         <geometry>
-          <mesh filename="package://robot_properties_kuka/meshes/stl/iiwa_link_3.stl" />
-        </geometry>
-        <material name="Orange"/>
-      </visual>
-      <collision>
-        <origin xyz="0 0 0" rpy="0 0 0"/>
-        <geometry>
-          <mesh filename="package://robot_properties_kuka/meshes/stl/iiwa_link_3.stl" />
+          <mesh filename="package://robot_properties_kuka/meshes/stl/iiwa_link_3.dae" scale="0.001 0.001 0.001"/>
+        </geometry>
+        <material name="Orange"/>
+      </visual>
+      <collision>
+        <origin xyz="0 0 0" rpy="0 0 0"/>
+        <geometry>
+          <mesh filename="package://robot_properties_kuka/meshes/stl/iiwa_link_3.dae" scale="0.001 0.001 0.001"/>
         </geometry>
         <material name="Orange"/>
@@ -173,12 +173,12 @@
         <origin xyz="0 0 0" rpy="0 0 0"/>
         <geometry>
-          <mesh filename="package://robot_properties_kuka/meshes/stl/iiwa_link_4.stl" />
-        </geometry>
-        <material name="Orange"/>
-      </visual>
-      <collision>
-        <origin xyz="0 0 0" rpy="0 0 0"/>
-        <geometry>
-          <mesh filename="package://robot_properties_kuka/meshes/stl/iiwa_link_4.stl" />
+          <mesh filename="package://robot_properties_kuka/meshes/stl/iiwa_link_4.dae" scale="0.001 0.001 0.001"/>
+        </geometry>
+        <material name="Orange"/>
+      </visual>
+      <collision>
+        <origin xyz="0 0 0" rpy="0 0 0"/>
+        <geometry>
+          <mesh filename="package://robot_properties_kuka/meshes/stl/iiwa_link_4.dae" scale="0.001 0.001 0.001"/>
         </geometry>
         <material name="Orange"/>
@@ -208,12 +208,12 @@
         <origin xyz="0 0 0" rpy="0 0 0"/>
         <geometry>
-          <mesh filename="package://robot_properties_kuka/meshes/stl/iiwa_link_5.stl" />
-        </geometry>
-        <material name="Orange"/>
-      </visual>
-      <collision>
-        <origin xyz="0 0 0" rpy="0 0 0"/>
-        <geometry>
-          <mesh filename="package://robot_properties_kuka/meshes/stl/iiwa_link_5.stl" />
+          <mesh filename="package://robot_properties_kuka/meshes/stl/iiwa_link_5.dae" scale="0.001 0.001 0.001"/>
+        </geometry>
+        <material name="Orange"/>
+      </visual>
+      <collision>
+        <origin xyz="0 0 0" rpy="0 0 0"/>
+        <geometry>
+          <mesh filename="package://robot_properties_kuka/meshes/stl/iiwa_link_5.dae" scale="0.001 0.001 0.001"/>
         </geometry>
         <material name="Orange"/>
@@ -243,12 +243,12 @@
         <origin xyz="0 0 0" rpy="0 0 0"/>
         <geometry>
-          <mesh filename="package://robot_properties_kuka/meshes/stl/iiwa_link_6.stl" />
-        </geometry>
-        <material name="Orange"/>
-      </visual>
-      <collision>
-        <origin xyz="0 0 0" rpy="0 0 0"/>
-        <geometry>
-          <mesh filename="package://robot_properties_kuka/meshes/stl/iiwa_link_6.stl" />
+          <mesh filename="package://robot_properties_kuka/meshes/stl/iiwa_link_6.dae" scale="0.001 0.001 0.001"/>
+        </geometry>
+        <material name="Orange"/>
+      </visual>
+      <collision>
+        <origin xyz="0 0 0" rpy="0 0 0"/>
+        <geometry>
+          <mesh filename="package://robot_properties_kuka/meshes/stl/iiwa_link_6.dae" scale="0.001 0.001 0.001"/>
         </geometry>
         <material name="Orange"/>
@@ -278,5 +278,5 @@
         <origin xyz="0 0 0" rpy="0 0 0"/>
         <geometry>
-          <mesh filename="package://robot_properties_kuka/meshes/stl/iiwa_link_7.stl" />
+          <mesh filename="package://robot_properties_kuka/meshes/stl/iiwa_link_7.dae" scale="0.001 0.001 0.001"/>
         </geometry>
         <material name="Grey"/>
@@ -285,5 +285,5 @@
         <origin xyz="0 0 0" rpy="0 0 0"/>
         <geometry>
-          <mesh filename="package://robot_properties_kuka/meshes/stl/iiwa_link_7.stl" />
+          <mesh filename="package://robot_properties_kuka/meshes/stl/iiwa_link_7.dae" scale="0.001 0.001 0.001"/>
         </geometry>
         <material name="Grey"/>

Commit message: corrected xacro (removed .dae and mesh scale)

File: src/robot_properties_kuka/robot_properties_kuka/xacro/iiwa.xacro (robot description, xacro)
@@ -26,5 +26,5 @@
         <origin xyz="0 0 0" rpy="0 0 0"/>
         <geometry>
-          <mesh filename="package://robot_properties_kuka/meshes/stl/iiwa_base.dae" scale="0.001 0.001 0.001"/>
+          <mesh filename="package://robot_properties_kuka/meshes/stl/iiwa_base.stl" />
         </geometry>
         <material name="Grey"/>
@@ -33,5 +33,5 @@
         <origin xyz="0 0 0" rpy="0 0 0"/>
         <geometry>
-          <mesh filename="package://robot_properties_kuka/meshes/stl/iiwa_base.dae" scale="0.001 0.001 0.001"/>
+          <mesh filename="package://robot_properties_kuka/meshes/stl/iiwa_base.stl" />
         </geometry>
         <material name="Grey"/>
@@ -68,12 +68,12 @@
         <origin xyz="0 0 0" rpy="0 0 0"/>
         <geometry>
-          <mesh filename="package://robot_properties_kuka/meshes/stl/iiwa_link_1.dae" scale="0.001 0.001 0.001"/>
-        </geometry>
-        <material name="Orange"/>
-      </visual>
-      <collision>
-        <origin xyz="0 0 0" rpy="0 0 0"/>
-        <geometry>
-          <mesh filename="package://robot_properties_kuka/meshes/stl/iiwa_link_1.dae" scale="0.001 0.001 0.001"/>
+          <mesh filename="package://robot_properties_kuka/meshes/stl/iiwa_link_1.stl" />
+        </geometry>
+        <material name="Orange"/>
+      </visual>
+      <collision>
+        <origin xyz="0 0 0" rpy="0 0 0"/>
+        <geometry>
+          <mesh filename="package://robot_properties_kuka/meshes/stl/iiwa_link_1.stl" />
         </geometry>
         <material name="Orange"/>
@@ -103,12 +103,12 @@
         <origin xyz="0 0 0" rpy="0 0 0"/>
         <geometry>
-          <mesh filename="package://robot_properties_kuka/meshes/stl/iiwa_link_2.dae" scale="0.001 0.001 0.001"/>
-        </geometry>
-        <material name="Orange"/>
-      </visual>
-      <collision>
-        <origin xyz="0 0 0" rpy="0 0 0"/>
-        <geometry>
-          <mesh filename="package://robot_properties_kuka/meshes/stl/iiwa_link_2.dae" scale="0.001 0.001 0.001"/>
+          <mesh filename="package://robot_properties_kuka/meshes/stl/iiwa_link_2.stl" />
+        </geometry>
+        <material name="Orange"/>
+      </visual>
+      <collision>
+        <origin xyz="0 0 0" rpy="0 0 0"/>
+        <geometry>
+          <mesh filename="package://robot_properties_kuka/meshes/stl/iiwa_link_2.stl" />
         </geometry>
         <material name="Orange"/>
@@ -138,12 +138,12 @@
         <origin xyz="0 0 0" rpy="0 0 0"/>
         <geometry>
-          <mesh filename="package://robot_properties_kuka/meshes/stl/iiwa_link_3.dae" scale="0.001 0.001 0.001"/>
-        </geometry>
-        <material name="Orange"/>
-      </visual>
-      <collision>
-        <origin xyz="0 0 0" rpy="0 0 0"/>
-        <geometry>
-          <mesh filename="package://robot_properties_kuka/meshes/stl/iiwa_link_3.dae" scale="0.001 0.001 0.001"/>
+          <mesh filename="package://robot_properties_kuka/meshes/stl/iiwa_link_3.stl" />
+        </geometry>
+        <material name="Orange"/>
+      </visual>
+      <collision>
+        <origin xyz="0 0 0" rpy="0 0 0"/>
+        <geometry>
+          <mesh filename="package://robot_properties_kuka/meshes/stl/iiwa_link_3.stl" />
         </geometry>
         <material name="Orange"/>
@@ -173,12 +173,12 @@
         <origin xyz="0 0 0" rpy="0 0 0"/>
         <geometry>
-          <mesh filename="package://robot_properties_kuka/meshes/stl/iiwa_link_4.dae" scale="0.001 0.001 0.001"/>
-        </geometry>
-        <material name="Orange"/>
-      </visual>
-      <collision>
-        <origin xyz="0 0 0" rpy="0 0 0"/>
-        <geometry>
-          <mesh filename="package://robot_properties_kuka/meshes/stl/iiwa_link_4.dae" scale="0.001 0.001 0.001"/>
+          <mesh filename="package://robot_properties_kuka/meshes/stl/iiwa_link_4.stl" />
+        </geometry>
+        <material name="Orange"/>
+      </visual>
+      <collision>
+        <origin xyz="0 0 0" rpy="0 0 0"/>
+        <geometry>
+          <mesh filename="package://robot_properties_kuka/meshes/stl/iiwa_link_4.stl" />
         </geometry>
         <material name="Orange"/>
@@ -208,12 +208,12 @@
         <origin xyz="0 0 0" rpy="0 0 0"/>
         <geometry>
-          <mesh filename="package://robot_properties_kuka/meshes/stl/iiwa_link_5.dae" scale="0.001 0.001 0.001"/>
-        </geometry>
-        <material name="Orange"/>
-      </visual>
-      <collision>
-        <origin xyz="0 0 0" rpy="0 0 0"/>
-        <geometry>
-          <mesh filename="package://robot_properties_kuka/meshes/stl/iiwa_link_5.dae" scale="0.001 0.001 0.001"/>
+          <mesh filename="package://robot_properties_kuka/meshes/stl/iiwa_link_5.stl" />
+        </geometry>
+        <material name="Orange"/>
+      </visual>
+      <collision>
+        <origin xyz="0 0 0" rpy="0 0 0"/>
+        <geometry>
+          <mesh filename="package://robot_properties_kuka/meshes/stl/iiwa_link_5.stl" />
         </geometry>
         <material name="Orange"/>
@@ -243,12 +243,12 @@
         <origin xyz="0 0 0" rpy="0 0 0"/>
         <geometry>
-          <mesh filename="package://robot_properties_kuka/meshes/stl/iiwa_link_6.dae" scale="0.001 0.001 0.001"/>
-        </geometry>
-        <material name="Orange"/>
-      </visual>
-      <collision>
-        <origin xyz="0 0 0" rpy="0 0 0"/>
-        <geometry>
-          <mesh filename="package://robot_properties_kuka/meshes/stl/iiwa_link_6.dae" scale="0.001 0.001 0.001"/>
+          <mesh filename="package://robot_properties_kuka/meshes/stl/iiwa_link_6.stl" />
+        </geometry>
+        <material name="Orange"/>
+      </visual>
+      <collision>
+        <origin xyz="0 0 0" rpy="0 0 0"/>
+        <geometry>
+          <mesh filename="package://robot_properties_kuka/meshes/stl/iiwa_link_6.stl" />
         </geometry>
         <material name="Orange"/>
@@ -278,5 +278,5 @@
         <origin xyz="0 0 0" rpy="0 0 0"/>
         <geometry>
-          <mesh filename="package://robot_properties_kuka/meshes/stl/iiwa_link_7.dae" scale="0.001 0.001 0.001"/>
+          <mesh filename="package://robot_properties_kuka/meshes/stl/iiwa_link_7.stl" />
         </geometry>
         <material name="Grey"/>
@@ -285,5 +285,5 @@
         <origin xyz="0 0 0" rpy="0 0 0"/>
         <geometry>
-          <mesh filename="package://robot_properties_kuka/meshes/stl/iiwa_link_7.dae" scale="0.001 0.001 0.001"/>
+          <mesh filename="package://robot_properties_kuka/meshes/stl/iiwa_link_7.stl" />
         </geometry>
         <material name="Grey"/>
@@ -311,5 +311,5 @@
         <origin rpy="0 0 0" xyz="0 0 0"/>
         <geometry>
-          <mesh filename="package://robot_properties_kuka/meshes/sphere.obj" scale="0.065 0.065 0.065"/>/>
+          <mesh filename="package://robot_properties_kuka/meshes/tennis_ball.obj" />
         </geometry>
         <material name="grey">
@@ -320,5 +320,5 @@
         <origin rpy="0 0 0" xyz="0 0 0"/>
         <geometry>
-          <mesh filename="package://robot_properties_kuka/meshes/sphere.obj" scale="0.065 0.065 0.065"/>/>
+          <mesh filename="package://robot_properties_kuka/meshes/tennis_ball.obj" />
         </geometry>
         <material name="grey">

Commit message: added tennis ball sized to 0.065 in blender + updated xacro

File: src/robot_properties_kuka/robot_properties_kuka/xacro/iiwa.xacro (robot description, xacro)
@@ -311,5 +311,5 @@
         <origin rpy="0 0 0" xyz="0 0 0"/>
         <geometry>
-          <mesh filename="package://robot_properties_kuka/meshes/tennis_ball.obj" />
+          <mesh filename="package://robot_properties_kuka/meshes/tennis_ball_smaller.obj" />
         </geometry>
         <material name="grey">
@@ -320,5 +320,5 @@
         <origin rpy="0 0 0" xyz="0 0 0"/>
         <geometry>
-          <mesh filename="package://robot_properties_kuka/meshes/tennis_ball.obj" />
+          <mesh filename="package://robot_properties_kuka/meshes/tennis_ball_smaller.obj" />
         </geometry>
         <material name="grey">

Commit message: fixed minor bug

File: src/robot_properties_kuka/robot_properties_kuka/xacro/iiwa.xacro (robot description, xacro)
@@ -49,5 +49,4 @@
       <parent link="iiwa_base"/>
       <child  link="L1"/>
-      <limit effort="30" velocity="1.0"/>
       <axis xyz="0 0 1"/>
       <limit lower="-2.96706" upper="2.96706" velocity="1.48353" effort="320"/>

Commit message: inertia fix for pybullet

File: src/robot_properties_kuka/robot_properties_kuka/xacro/iiwa.xacro (robot description, xacro)
@@ -167,5 +167,5 @@
         <origin xyz="0 0.067 0.034" rpy="0 0 0"/>
         <mass value="2.61155"/>
-        <inertia ixx="0.03844"  ixy="0.00088"  ixz="-0.00112" iyy="0.01144" iyz="-0.00111" izz="0.04988" />
+        <inertia ixx="0.03844"  ixy="0.00088"  ixz="-0.00112" iyy="0.01144" iyz="-0.00111" izz="0.04958" />
       </inertial>
       <visual>
@@ -272,5 +272,5 @@
         <origin xyz="0 0 0.02" rpy="0 0 0"/>
         <mass value="0.35432"/>
-        <inertia ixx="0.00795"  ixy="0.00022"  ixz="-0.00029" iyy="0.01089" iyz="-0.00029" izz="0.00294" />
+        <inertia ixx="0.00795"  ixy="0.00022"  ixz="-0.00029" iyy="0.01083" iyz="-0.00029" izz="0.00294" />
       </inertial>
       <visual>
