Commit message: added demo file meshcat + assembled ft sensor mount piece in urdf

File: src/robot_properties_kuka/robot_properties_kuka/xacro/iiwa.xacro (robot description, xacro)
@@ -292,7 +292,7 @@
     <joint name="EE" type="fixed">
       <parent link="L7"/>
-      <child link="contact"/>
+      <child link="assembled_ee"/>
       <!-- Joint placement -->
-      <origin rpy="0 0 0" xyz="0 0.0 0.04"/>
+      <origin rpy="1.57079632679 0 0" xyz="0 0 0.04"/>
       <!-- Limits (usefull?) -->
       <limit effort="1000" lower="-10" upper="10" velocity="1000"/>
@@ -300,4 +300,41 @@
       <dynamics damping="0.0" friction="0.0"/>
     </joint>
+    <!-- assembled_ee -->
+    <link name="assembled_ee">
+      <inertial>
+        <origin rpy="0 0 0" xyz="0 0.01892 0"/>
+        <mass value="0.07937"/>
+        <inertia ixx="0.000132912903" ixy="0" ixz="0.00000007" iyy="0.000067699" iyz="0.0000000017" izz="0.000128095503"/>
+      </inertial>
+      <visual>
+        <origin rpy="0 0 0" xyz="0 0 0"/>
+        <geometry>
+          <mesh scale="0.001 0.001 0.001" filename="package://robot_properties_kuka/meshes/stl/assembled_ee.stl" />
+        </geometry>
+        <material name="White">
+          <color rgba="0.9 0.9 0.9 0.9"/>
+        </material>
+      </visual>
+      <collision>
+        <origin rpy="0 0 0" xyz="0 0 0"/>
+        <geometry>
+          <mesh scale="0.001 0.001 0.001" filename="package://robot_properties_kuka/meshes/stl/assembled_ee.stl" />
+        </geometry>
+        <material name="White">
+          <color rgba="0.9 0.9 0.9 0.9"/>
+        </material>
+      </collision>
+    </link>
+    <!-- fixed joint assembled_ee <=> soft ball tip -->
+    <joint name="ee_to_contact_joint" type="fixed">
+      <parent link="assembled_ee"/>
+      <child link="contact"/>
+      <!-- Joint placement -->
+      <origin rpy="0 0 0" xyz="0 0.1 0"/>
+      <!-- Limits (usefull?) -->
+      <limit effort="1000" lower="-10" upper="10" velocity="1000"/>
+      <!-- pybullet simulation parameters -->
+      <dynamics damping="0.0" friction="0.0"/>
+    </joint>
     <!-- CONTACT (modeled by a tennis ball) -->
     <link name="contact">
@@ -312,6 +349,6 @@
           <mesh filename="package://robot_properties_kuka/meshes/tennis_ball_smaller.obj" />
         </geometry>
-        <material name="grey">
-          <color rgba="0.8 0.8 0.8 1.0"/>
+        <material name="Green">
+          <color rgba="0. 0.8 0. 0.8"/>
         </material>
       </visual>
@@ -321,6 +358,6 @@
           <mesh filename="package://robot_properties_kuka/meshes/tennis_ball_smaller.obj" />
         </geometry>
-        <material name="grey">
-          <color rgba="0.8 0.8 0.8 1.0"/>
+        <material name="Green">
+          <color rgba="0. 0.8 0. 0.8"/>
         </material>
       </collision>

Commit message: fixed frame of tennis ball to have z as normal

File: src/robot_properties_kuka/robot_properties_kuka/xacro/iiwa.xacro (robot description, xacro)
@@ -331,5 +331,5 @@
       <child link="contact"/>
       <!-- Joint placement -->
-      <origin rpy="0 0 0" xyz="0 0.1 0"/>
+      <origin rpy="-1.57079632679 0 0" xyz="0 0.1 0"/>
       <!-- Limits (usefull?) -->
       <limit effort="1000" lower="-10" upper="10" velocity="1000"/>

Commit message: replaced tennis ball by soft polystyrene ball in urdf

File: src/robot_properties_kuka/robot_properties_kuka/xacro/iiwa.xacro (robot description, xacro)
@@ -313,5 +313,5 @@
         </geometry>
         <material name="White">
-          <color rgba="0.9 0.9 0.9 0.9"/>
+          <color rgba="0.9 0.9 0.9 0.7"/>
         </material>
       </visual>
@@ -322,5 +322,5 @@
         </geometry>
         <material name="White">
-          <color rgba="0.9 0.9 0.9 0.9"/>
+          <color rgba="0.9 0.9 0.9 0.7"/>
         </material>
       </collision>
@@ -331,5 +331,5 @@
       <child link="contact"/>
       <!-- Joint placement -->
-      <origin rpy="-1.57079632679 0 0" xyz="0 0.1 0"/>
+      <origin rpy="-1.57079632679 0 0" xyz="0 0.06 0"/>
       <!-- Limits (usefull?) -->
       <limit effort="1000" lower="-10" upper="10" velocity="1000"/>
@@ -337,15 +337,16 @@
       <dynamics damping="0.0" friction="0.0"/>
     </joint>
-    <!-- CONTACT (modeled by a tennis ball) -->
+    <!-- CONTACT (modeled by a soft polystyrene ball) -->
     <link name="contact">
       <inertial>
         <origin rpy="0 0 0" xyz="0 0 0.0"/>
-        <mass value="0.057"/>
-        <inertia ixx="0.0000354" ixy="0.0" ixz="0.0" iyy="0.0000354" iyz="0.0" izz="0.0000354"/>
+        <mass value="0.014"/>
+        <inertia ixx="0.00000126" ixy="0.0" ixz="0.0" iyy="0.00000126" iyz="0.0" izz="0.00000126"/>
       </inertial>
       <visual>
         <origin rpy="0 0 0" xyz="0 0 0"/>
         <geometry>
-          <mesh filename="package://robot_properties_kuka/meshes/tennis_ball_smaller.obj" />
+          <sphere radius="0.015" />
+          <!-- <mesh filename="package://robot_properties_kuka/meshes/tennis_ball_smaller.obj" /> -->
         </geometry>
         <material name="Green">
@@ -356,5 +357,6 @@
         <origin rpy="0 0 0" xyz="0 0 0"/>
         <geometry>
-          <mesh filename="package://robot_properties_kuka/meshes/tennis_ball_smaller.obj" />
+          <sphere radius="0.015" />
+          <!-- <mesh filename="package://robot_properties_kuka/meshes/tennis_ball_smaller.obj" /> -->
         </geometry>
         <material name="Green">

Commit message: created 3 different urdfs: no endeff, ft_sensor+shell and ft_sensor+ball transfer

File: src/robot_properties_kuka/robot_properties_kuka/xacro/iiwa.xacro (robot description, xacro)
@@ -292,7 +292,7 @@
     <joint name="EE" type="fixed">
       <parent link="L7"/>
-      <child link="assembled_ee"/>
+      <child link="contact"/>
       <!-- Joint placement -->
-      <origin rpy="1.57079632679 0 0" xyz="0 0 0.04"/>
+      <origin rpy="0 0 0" xyz="0 0.0 0.04"/>
       <!-- Limits (usefull?) -->
       <limit effort="1000" lower="-10" upper="10" velocity="1000"/>
@@ -300,18 +300,18 @@
       <dynamics damping="0.0" friction="0.0"/>
     </joint>
-    <!-- assembled_ee -->
-    <link name="assembled_ee">
-      <inertial>
-        <origin rpy="0 0 0" xyz="0 0.01892 0"/>
-        <mass value="0.07937"/>
-        <inertia ixx="0.000132912903" ixy="0" ixz="0.00000007" iyy="0.000067699" iyz="0.0000000017" izz="0.000128095503"/>
+    <!-- CONTACT (modeled by a tennis ball) -->
+    <link name="contact">
+      <inertial>
+        <origin rpy="0 0 0" xyz="0 0 0.0"/>
+        <mass value="0.057"/>
+        <inertia ixx="0.0000354" ixy="0.0" ixz="0.0" iyy="0.0000354" iyz="0.0" izz="0.0000354"/>
       </inertial>
       <visual>
         <origin rpy="0 0 0" xyz="0 0 0"/>
         <geometry>
-          <mesh scale="0.001 0.001 0.001" filename="package://robot_properties_kuka/meshes/stl/assembled_ee.stl" />
-        </geometry>
-        <material name="White">
-          <color rgba="0.9 0.9 0.9 0.7"/>
+          <mesh filename="package://robot_properties_kuka/meshes/tennis_ball_smaller.obj" />
+        </geometry>
+        <material name="grey">
+          <color rgba="0.8 0.8 0.8 1.0"/>
         </material>
       </visual>
@@ -319,47 +319,8 @@
         <origin rpy="0 0 0" xyz="0 0 0"/>
         <geometry>
-          <mesh scale="0.001 0.001 0.001" filename="package://robot_properties_kuka/meshes/stl/assembled_ee.stl" />
-        </geometry>
-        <material name="White">
-          <color rgba="0.9 0.9 0.9 0.7"/>
-        </material>
-      </collision>
-    </link>
-    <!-- fixed joint assembled_ee <=> soft ball tip -->
-    <joint name="ee_to_contact_joint" type="fixed">
-      <parent link="assembled_ee"/>
-      <child link="contact"/>
-      <!-- Joint placement -->
-      <origin rpy="-1.57079632679 0 0" xyz="0 0.06 0"/>
-      <!-- Limits (usefull?) -->
-      <limit effort="1000" lower="-10" upper="10" velocity="1000"/>
-      <!-- pybullet simulation parameters -->
-      <dynamics damping="0.0" friction="0.0"/>
-    </joint>
-    <!-- CONTACT (modeled by a soft polystyrene ball) -->
-    <link name="contact">
-      <inertial>
-        <origin rpy="0 0 0" xyz="0 0 0.0"/>
-        <mass value="0.014"/>
-        <inertia ixx="0.00000126" ixy="0.0" ixz="0.0" iyy="0.00000126" iyz="0.0" izz="0.00000126"/>
-      </inertial>
-      <visual>
-        <origin rpy="0 0 0" xyz="0 0 0"/>
-        <geometry>
-          <sphere radius="0.015" />
-          <!-- <mesh filename="package://robot_properties_kuka/meshes/tennis_ball_smaller.obj" /> -->
-        </geometry>
-        <material name="Green">
-          <color rgba="0. 0.8 0. 0.8"/>
-        </material>
-      </visual>
-      <collision>
-        <origin rpy="0 0 0" xyz="0 0 0"/>
-        <geometry>
-          <sphere radius="0.015" />
-          <!-- <mesh filename="package://robot_properties_kuka/meshes/tennis_ball_smaller.obj" /> -->
-        </geometry>
-        <material name="Green">
-          <color rgba="0. 0.8 0. 0.8"/>
+          <mesh filename="package://robot_properties_kuka/meshes/tennis_ball_smaller.obj" />
+        </geometry>
+        <material name="grey">
+          <color rgba="0.8 0.8 0.8 1.0"/>
         </material>
       </collision>
