Commit message: changed ball transfer stl to obj & fixed bad inertia props of kuka_to_sensor_mount

File: src/robot_properties_kuka/robot_properties_kuka/xacro/iiwa_ft_sensor_ball.xacro (robot description, xacro)
@@ -305,5 +305,5 @@
         <origin rpy="0 0 0" xyz="0 0.452 0"/>
         <mass value="0.042647"/>
-        <inertia ixx="0.0000014879" ixy="0.0" ixz="0.0" iyy="0.0002270" iyz="0.0000000017" izz="0.0001171"/>
+        <inertia ixx="0.0000014879" ixy="0.0" ixz="0.0" iyy="0.0001171" iyz="0.0" izz="0.0001171"/>
       </inertial>
       <visual>
@@ -421,15 +421,14 @@
         <origin rpy="0 0 0" xyz="0 0 0"/>
         <geometry>
-          <!-- <mesh scale="0.03937007874 0.03937007874 0.03937007874" filename="package://robot_properties_kuka/meshes/stl/5674K57_flange_mount_ball_transfer.stl" /> -->
-          <mesh scale="0.0254 0.0254 0.0254" filename="package://robot_properties_kuka/meshes/stl/5674K57_flange_mount_ball_transfer.stl" />
-        </geometry>
-        <material name="grey">
-          <color rgba="0.8 0.8 0.8 1.0"/>
-        </material>
-      </visual>
-      <collision>
-        <origin rpy="0 0 0" xyz="0 0 0"/>
-        <geometry>
-          <mesh scale="0.0254 0.0254 0.0254" filename="package://robot_properties_kuka/meshes/stl/5674K57_flange_mount_ball_transfer.stl" />
+          <mesh scale="0.0254 0.0254 0.0254" filename="package://robot_properties_kuka/meshes/obj/5674K57_flange_mount_ball_transfer.obj" />
+        </geometry>
+        <material name="grey">
+          <color rgba="0.8 0.8 0.8 1.0"/>
+        </material>
+      </visual>
+      <collision>
+        <origin rpy="0 0 0" xyz="0 0 0"/>
+        <geometry>
+          <mesh scale="0.0254 0.0254 0.0254" filename="package://robot_properties_kuka/meshes/obj/5674K57_flange_mount_ball_transfer.obj" />
         </geometry>
         <material name="grey">

Commit message: renamed last fixed joint before contact frame to EE

File: src/robot_properties_kuka/robot_properties_kuka/xacro/iiwa_ft_sensor_ball.xacro (robot description, xacro)
@@ -289,6 +289,6 @@
       </collision>
     </link>
-    <!-- EE -->
-    <joint name="EE" type="fixed">
+    <!-- kuka_to_sensor_mount_joint -->
+    <joint name="kuka_to_sensor_mount_joint" type="fixed">
       <parent link="L7"/>
       <child link="kuka_to_sensor_mount"/>
@@ -401,5 +401,5 @@
     </link>
     <!-- fixed joint ft_sensor <=> case_mount -->
-    <joint name="mount_to_case_joint" type="fixed">
+    <joint name="EE" type="fixed">
       <parent link="sensor_to_case_mount"/>
       <child link="contact"/>
@@ -436,4 +436,9 @@
         </material>
       </collision>
+      <!-- Bullet specific paramters -->
+      <contact>
+        <lateral_friction value="0.0"/>
+        <restitution value="0.5"/>
+      </contact>
     </link>
     <!--Extensions -->

File: src/robot_properties_kuka/robot_properties_kuka/xacro/iiwa_ft_sensor_shell.xacro (robot description, xacro)
@@ -289,6 +289,6 @@
       </collision>
     </link>
-    <!-- EE -->
-    <joint name="EE" type="fixed">
+    <!-- kuka_to_assembled_ee_joint -->
+    <joint name="kuka_to_assembled_ee_joint" type="fixed">
       <parent link="L7"/>
       <child link="assembled_ee"/>
@@ -327,5 +327,5 @@
     </link>
     <!-- fixed joint assembled_ee <=> soft ball tip -->
-    <joint name="ee_to_contact_joint" type="fixed">
+    <joint name="EE" type="fixed">
       <parent link="assembled_ee"/>
       <child link="contact"/>

Commit message: fixed inertial kuka_to_sensor_mount

File: src/robot_properties_kuka/robot_properties_kuka/xacro/iiwa_ft_sensor_ball.xacro (robot description, xacro)
@@ -303,5 +303,5 @@
     <link name="kuka_to_sensor_mount">
       <inertial>
-        <origin rpy="0 0 0" xyz="0 0.452 0"/>
+        <origin rpy="0 0 0" xyz="0 0 0"/>
         <mass value="0.042647"/>
         <inertia ixx="0.0000014879" ixy="0.0" ixz="0.0" iyy="0.0001171" iyz="0.0" izz="0.0001171"/>

Commit message: fixed contact frame orientation for flange mount ball transfer urdf + added cad frame name as attribute of the config

File: src/robot_properties_kuka/robot_properties_kuka/xacro/iiwa_ft_sensor_ball.xacro (robot description, xacro)
@@ -289,10 +289,10 @@
       </collision>
     </link>
-    <!-- kuka_to_sensor_mount_joint -->
-    <joint name="kuka_to_sensor_mount_joint" type="fixed">
+    <!-- kuka_to_ee_joint -->
+    <joint name="kuka_to_ee_joint" type="fixed">
       <parent link="L7"/>
       <child link="kuka_to_sensor_mount"/>
       <!-- Joint placement -->
-      <origin rpy="1.57079632679 0 0" xyz="0 0.0 0.045"/>
+      <origin rpy="1.57079632679 0 0" xyz="0 0 0.045"/>
       <!-- Limits (usefull?) -->
       <limit effort="1000" lower="-10" upper="10" velocity="1000"/>
@@ -331,5 +331,5 @@
       <child link="ft_sensor"/>
       <!-- Joint placement -->
-      <origin rpy="-1.57079632679 0 0" xyz="0 0.018 0.0"/>
+      <origin rpy="-1.57079632679 0 0" xyz="0 0.01795 0"/>
       <!-- Limits (usefull?) -->
       <limit effort="1000" lower="-10" upper="10" velocity="1000"/>
@@ -340,5 +340,5 @@
     <link name="ft_sensor">
       <inertial>
-        <origin rpy="0 0 0" xyz="0 0 0"/>
+        <origin rpy="0 0 0" xyz="0 0 0.00785"/>
         <mass value="0.091"/>
         <inertia ixx="0.0000133864" ixy="0" ixz="0" iyy="0.0000133864" iyz="0" izz="0.000023034375"/>
@@ -368,5 +368,5 @@
       <child link="sensor_to_case_mount"/>
       <!-- Joint placement -->
-      <origin rpy="1.57079632679 0 0" xyz="0 0.0 0.008"/>
+      <origin rpy="1.57079632679 0 0" xyz="0 0 0.00785"/>
       <!-- Limits (usefull?) -->
       <limit effort="1000" lower="-10" upper="10" velocity="1000"/>
@@ -401,9 +401,9 @@
     </link>
     <!-- fixed joint ft_sensor <=> case_mount -->
-    <joint name="EE" type="fixed">
+    <joint name="case_mount_to_ball_transfer" type="fixed">
       <parent link="sensor_to_case_mount"/>
-      <child link="contact"/>
+      <child link="ball_transfer"/>
       <!-- Joint placement -->
-      <origin rpy="0 1.57079632679 0" xyz="0 0.003 0.0"/>
+      <origin rpy="0 1.57079632679 0" xyz="0 0.0025 0.0"/>
       <!-- Limits (usefull?) -->
       <limit effort="1000" lower="-10" upper="10" velocity="1000"/>
@@ -411,6 +411,6 @@
       <dynamics damping="0.0" friction="0.0"/>
     </joint>
-    <!-- contact = flang mount ball transfer-->
-    <link name="contact">
+    <!-- flang mount ball transfer-->
+    <link name="ball_transfer">
       <inertial>
         <origin rpy="0 0 0" xyz="0 0.000916 0"/>
@@ -442,4 +442,48 @@
       </contact>
     </link>
+    <!-- fixed joint assembled_ee <=> soft ball tip -->
+    <joint name="EE" type="fixed">
+      <parent link="ball_transfer"/>
+      <child link="contact"/>
+      <!-- Joint placement -->
+      <origin rpy="0 -1.57079632679 -1.57079632679" xyz="0 0.0254 0"/>
+      <!-- Limits (usefull?) -->
+      <limit effort="1000" lower="-10" upper="10" velocity="1000"/>
+      <!-- pybullet simulation parameters -->
+      <dynamics damping="0.0" friction="0.0"/>
+    </joint>
+    <!-- CONTACT (modeled by a soft polystyrene ball) -->
+    <link name="contact">
+      <inertial>
+        <origin rpy="0 0 0" xyz="0 0 -0.00873"/>
+        <mass value="0.014"/>
+        <inertia ixx="0.00000126" ixy="0.0" ixz="0.0" iyy="0.00000126" iyz="0.0" izz="0.00000126"/>
+      </inertial>
+      <visual>
+        <origin rpy="0 0 0" xyz="0 0 -0.00873"/>
+        <geometry>
+          <sphere radius="0.00873" />
+          <!-- <mesh filename="package://robot_properties_kuka/meshes/tennis_ball_smaller.obj" /> -->
+        </geometry>
+        <material name="Green">
+          <color rgba="0. 0.8 0. 0.8"/>
+        </material>
+      </visual>
+      <collision>
+        <origin rpy="0 0 0" xyz="0 0 -0.00873"/>
+        <geometry>
+          <sphere radius="0.00873" />
+          <!-- <mesh filename="package://robot_properties_kuka/meshes/tennis_ball_smaller.obj" /> -->
+        </geometry>
+        <material name="Green">
+          <color rgba="0. 0.8 0. 0.8"/>
+        </material>
+      </collision>
+      <!-- Bullet specific paramters -->
+      <contact>
+        <lateral_friction value="1.0"/>
+        <restitution value="0.5"/>
+      </contact>
+    </link>
     <!--Extensions -->
     <xacro:iiwa_gazebo robot_name="KUKAiiwa14"/>

File: src/robot_properties_kuka/robot_properties_kuka/xacro/iiwa_ft_sensor_shell.xacro (robot description, xacro)
@@ -289,10 +289,10 @@
       </collision>
     </link>
-    <!-- kuka_to_assembled_ee_joint -->
-    <joint name="kuka_to_assembled_ee_joint" type="fixed">
+    <!-- kuka_to_ee_joint -->
+    <joint name="kuka_to_ee_joint" type="fixed">
       <parent link="L7"/>
       <child link="assembled_ee"/>
       <!-- Joint placement -->
-      <origin rpy="1.57079632679 0 0" xyz="0 0 0.04"/>
+      <origin rpy="1.57079632679 0 0" xyz="0 0 0.045"/>
       <!-- Limits (usefull?) -->
       <limit effort="1000" lower="-10" upper="10" velocity="1000"/>

Commit message: changed ft_sensor name to ft_sensor_link to avoid clash with manually added OP frame + fixed contact origin + fixed friction coef

File: src/robot_properties_kuka/robot_properties_kuka/xacro/iiwa_ft_sensor_ball.xacro (robot description, xacro)
@@ -329,5 +329,5 @@
     <joint name="mount_to_sensor_joint" type="fixed">
       <parent link="kuka_to_sensor_mount"/>
-      <child link="ft_sensor"/>
+      <child link="ft_sensor_link"/>
       <!-- Joint placement -->
       <origin rpy="-1.57079632679 0 0" xyz="0 0.01795 0"/>
@@ -337,6 +337,6 @@
       <dynamics damping="0.0" friction="0.0"/>
     </joint>
-    <!-- ft_sensor (Schunk) -->
-    <link name="ft_sensor">
+    <!-- ft_sensor_link (Schunk) -->
+    <link name="ft_sensor_link">
       <inertial>
         <origin rpy="0 0 0" xyz="0 0 0.00785"/>
@@ -363,7 +363,7 @@
       </collision>
     </link>
-    <!-- fixed joint ft_sensor <=> case_mount -->
+    <!-- fixed joint ft_sensor_link <=> case_mount -->
     <joint name="sensor_to_case_joint" type="fixed">
-      <parent link="ft_sensor"/>
+      <parent link="ft_sensor_link"/>
       <child link="sensor_to_case_mount"/>
       <!-- Joint placement -->
@@ -400,5 +400,5 @@
       </collision>
     </link>
-    <!-- fixed joint ft_sensor <=> case_mount -->
+    <!-- fixed joint sensor_to_case_mount <=> ball_transfer -->
     <joint name="case_mount_to_ball_transfer" type="fixed">
       <parent link="sensor_to_case_mount"/>
@@ -447,5 +447,5 @@
       <child link="contact"/>
       <!-- Joint placement -->
-      <origin rpy="0 -1.57079632679 -1.57079632679" xyz="0 0.0254 0"/>
+      <origin rpy="0 -1.57079632679 -1.57079632679" xyz="0 0.027 0"/>
       <!-- Limits (usefull?) -->
       <limit effort="1000" lower="-10" upper="10" velocity="1000"/>
@@ -482,5 +482,5 @@
       <!-- Bullet specific paramters -->
       <contact>
-        <lateral_friction value="1.0"/>
+        <lateral_friction value="0."/>
         <restitution value="0.5"/>
       </contact>
